File: kiln.kicad_sch (KiCad schematic)
At the start: 0 parts

Commit message: sch progress
Other:
- sheet MainControler ports: added DataFromSafty, DataToSafty, Fault; removed none
- sheet Power ports: added 8V; removed none
- sheet SaftyProcessor ports: added 8V, DataFromSafty, DataGnd, DataToSafty, Fault; removed none

Commit message: more sch updates
Other:
- sheet Power ports: added PwrGnd; removed Gnd
Changed lines of the file:
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@@
+	(wire
+		(pts
+			(xy 102.87 92.71) (xy 102.87 95.25)
+		)
+		(stroke
+			(width 0)
+			(type default)
+		)
+	)
+	(wire
+		(pts
+			(xy 111.76 139.7) (xy 111.76 149.86)
+		)
+		(stroke
+			(width 0)
+			(type default)
+		)
+	)
 	(wire
 		(pts
@@
 	(wire
 		(pts
-			(xy 111.76 139.7) (xy 111.76 149.86)
-		)
-		(stroke
-			(width 0)
-			(type default)
-		)
-	)
-	(wire
-		(pts
 			(xy 109.22 105.41) (xy 123.19 105.41)
 		)
@@
 		(pts
 			(xy 106.68 93.98) (xy 106.68 95.25)
-		)
-		(stroke
-			(width 0)
-			(type default)
-		)
-	)
-	(wire
-		(pts
-			(xy 102.87 92.71) (xy 102.87 95.25)
 		)
 		(stroke
@@
 			)
 		)
-		(pin "3.3V" passive
-			(at 132.08 95.25 90)
-			(effects
-				(font
-					(size 1.27 1.27)
-				)
-				(justify right)
-			)
-		)
-		(pin "5V" passive
-			(at 134.62 95.25 90)
-			(effects
-				(font
-					(size 1.27 1.27)
-				)
-				(justify right)
-			)
-		)
 		(pin "GND" passive
 			(at 133.35 118.11 270)
@@
 			)
 		)
-		(pin "12V" passive
-			(at 129.54 95.25 90)
-			(effects
-				(font
-					(size 1.27 1.27)
-				)
-				(justify right)
-			)
-		)
 		(pin "DataFromSafty" input
 			(at 123.19 105.41 180)
@@
 				)
 				(justify left)
+			)
+		)
+		(pin "3.3V" input
+			(at 134.62 95.25 90)
+			(effects
+				(font
+					(size 1.27 1.27)
+				)
+				(justify right)
+			)
+		)
+		(pin "5V" input
+			(at 132.08 95.25 90)
+			(effects
+				(font
+					(size 1.27 1.27)
+				)
+				(justify right)
+			)
+		)
+		(pin "12V" input
+			(at 129.54 95.25 90)
+			(effects
+				(font
+					(size 1.27 1.27)
+				)
+				(justify right)
 			)
 		)
@@
 			)
 		)
-		(pin "12V" passive
-			(at 106.68 95.25 90)
-			(effects
-				(font
-					(size 1.27 1.27)
-				)
-				(justify right)
-			)
-		)
 		(pin "GND" passive
 			(at 106.68 119.38 270)
@@
 			)
 		)
-		(pin "8V" passive
-			(at 102.87 95.25 90)
-			(effects
-				(font
-					(size 1.27 1.27)
-				)
-				(justify right)
-			)
-		)
 		(pin "DataGnd" passive
 			(at 101.6 119.38 270)
@@
 		(pin "Fault" input
 			(at 109.22 102.87 0)
+			(effects
+				(font
+					(size 1.27 1.27)
+				)
+				(justify right)
+			)
+		)
+		(pin "8V" input
+			(at 102.87 95.25 90)
+			(effects
+				(font
+					(size 1.27 1.27)
+				)
+				(justify right)
+			)
+		)
+		(pin "12V" input
+			(at 106.68 95.25 90)
 			(effects
 				(font
@@
 			)
 		)
-		(pin "3.3V" passive
+		(pin "3.3V" output
 			(at 116.84 149.86 90)
 			(effects
@@
 			)
 		)
-		(pin "5V" passive
+		(pin "5V" output
 			(at 114.3 149.86 90)
 			(effects
@@
 			)
 		)
-		(pin "Gnd" passive
+		(pin "8V" output
+			(at 107.95 149.86 90)
+			(effects
+				(font
+					(size 1.27 1.27)
+				)
+				(justify right)
+			)
+		)
+		(pin "12V" output
+			(at 111.76 149.86 90)
+			(effects
+				(font
+					(size 1.27 1.27)
+				)
+				(justify right)
+			)
+		)
+		(pin "PwrGnd" passive
 			(at 114.3 163.83 270)
 			(effects
@@
 			)
 		)
-		(pin "12V" passive
-			(at 111.76 149.86 90)
-			(effects
-				(font
-					(size 1.27 1.27)
-				)
-				(justify right)
-			)
-		)
-		(pin "8V" passive
-			(at 107.95 149.86 90)
-			(effects
-				(font
-					(size 1.27 1.27)
-				)
-				(justify right)
-			)
-		)

Commit message: sch progress
Other:
- removed sheet Power
- added sheet MainRegulators (Regulators.kicad_sch)
- added sheet SaftyRegulators (Regulators.kicad_sch)
- sheet MainControler ports: added Gnd; removed GND
- sheet SaftyProcessor ports: added 3.3V, 5V, Gnd, MainProcessorDataGnd; removed 8V, DataGnd, GND
- note removed: "https://www.sparkfun.com/sparkfun-transceiver-breakout-rs-485.html"
