File: kiln.kicad_sch (KiCad schematic)
At the start: 0 parts

Commit message: progress
Other:
- sheet MainControler ports: added none; removed 5V
- sheet MainRegulators ports: added none; removed 5V
- sheet SaftyProcessor ports: added none; removed 5V
- sheet SaftyRegulators ports: added none; removed 5V
Changed lines of the file:
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@@
-	(wire
-		(pts
-			(xy 128.27 95.25) (xy 128.27 81.28)
-		)
-		(stroke
-			(width 0)
-			(type default)
-		)
-	)
 	(wire
 		(pts
@@
 	(wire
 		(pts
-			(xy 128.27 81.28) (xy 152.4 81.28)
-		)
-		(stroke
-			(width 0)
-			(type default)
-		)
-	)
-	(wire
-		(pts
-			(xy 92.71 95.25) (xy 92.71 82.55)
-		)
-		(stroke
-			(width 0)
-			(type default)
-		)
-	)
-	(wire
-		(pts
 			(xy 138.43 123.19) (xy 149.86 123.19)
 		)
@@
 		(pts
 			(xy 149.86 88.9) (xy 152.4 88.9)
-		)
-		(stroke
-			(width 0)
-			(type default)
-		)
-	)
-	(wire
-		(pts
-			(xy 92.71 82.55) (xy 73.66 82.55)
 		)
 		(stroke
@@
 		(pin "3.3V" input
 			(at 90.17 95.25 90)
-			(effects
-				(font
-					(size 1.27 1.27)
-				)
-				(justify right)
-			)
-		)
-		(pin "5V" input
-			(at 92.71 95.25 90)
 			(effects
 				(font
@@
 			)
 		)
-		(pin "5V" output
-			(at 152.4 81.28 180)
-			(effects
-				(font
-					(size 1.27 1.27)
-				)
-				(justify left)
-			)
-		)
 		(pin "12V" output
 			(at 152.4 77.47 180)
@@
 			)
 		)
-		(pin "5V" output
-			(at 73.66 82.55 0)
-			(effects
-				(font
-					(size 1.27 1.27)
-				)
-				(justify right)
-			)
-		)
 		(pin "12V" output
 			(at 73.66 78.74 0)
@@
 			(effects
 				(font
-					(size 1.27 1.27)
-				)
-				(justify right)
-			)
-		)
-		(pin "5V" input
-			(at 128.27 95.25 90)
-			(effects
-				(font

Commit message: sch looks prety good
Other:
- sheet MainRegulators renamed MainRegulator
- sheet SaftyRegulators renamed SaftyRegulator
- added sheet 5V Regulator (5V_Regulator.kicad_sch)
- sheet MainControler ports: added 5V; removed none
- sheet MainRegulator ports: added PGood; removed none
- sheet SaftyRegulator ports: added PGood; removed none
