File: MainControler.kicad_sch (KiCad schematic)
At the start: 27 parts, among them J5 1935161, J6 1935161, SW2 SW_Push, U5 TXS0108EPW, U6 TXS0108EPW, U7 MAX3490xSA

Commit message: sch progress
Parts:
- removed C12: 0.001uf, Capacitor_SMD:C_0402_1005Metric, symbol Device:C
- added C11: 0.01uf, Capacitor_SMD:C_0402_1005Metric, symbol Device:C
- added R29: 1k, Resistor_SMD:R_0402_1005Metric, symbol Device:R
- renumbered J5 to J6, J6 to J7, R13 to R19, R15 to R20, R14 to R21, R16 to R22, R17 to R23, R18 to R24, R19 to R25, R20 to R26, R21 to R27, R23 to R28, R22 to R30, U7 to U10, U5 to U8, U6 to U9
Connections:
- net 5V_Main: now also R29.2
- net GND_Main: now also C11.2
- net UartRx: now also A2.5 (D2); no longer A2.2 (D0/RX)
- net UartTx: now also A2.6 (D3); no longer A2.1 (D1/TX)
- net saftyRelay: now also A2.7 (D4); no longer A2.5 (D2)
- net thermoDrdy: now also A2.9 (D6); no longer A2.7 (D4)
- net thermoFault: now also A2.8 (D5); no longer A2.6 (D3)
- net at A2.28 (~{RESET}), R28.1, SW2.2: now also C11.1
- net Fault: now reaches A2.22 (A3)
- net DataToSafty: now reaches A2.23 (A4)
- net DataFromSafty: now reaches A2.24 (A5)
- net DataFromSafty: now also R29.1
Other:
- moved on the sheet: A2, R19, R20, R21, R22, R23, R24, R25, R26, R27, R28, SW2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

Commit message: more sch updates
Parts:
- added R26, R29, R30, R31, R32: 0, Resistor_SMD:R_0805_2012Metric, symbol Device:R
- renumbered D9 to D10, D10 to D11, D11 to D12, D12 to D13, D13 to D14, D14 to D15, D15 to D16, D16 to D17, R26 to R27, R27 to R28, R28 to R33, R29 to R34, R30 to R35
Connections:
- net 3.3V_Main: now also R26.1, R31.1, R32.2
- net 5V_Main: now also R29.2, R30.1; no longer U8.19 (VCCB), U9.19 (VCCB)
- net Relay1: now also A2.19 (A0)
- net Relay2: now also A2.20 (A1)
- net Relay3: now also A2.21 (A2)
- net at A2.17 (3V3): now also R31.2
- net saftyRelay: no longer names the net of A2.7 (D4)
- new net: R30.2, R32.1, U9.19 (VCCB)
- new net: R26.2, R29.1, U8.19 (VCCB)
Other:
- sheet SSD ports: added RelayGND; removed GND
- sheet SSD1 ports: added RelayGND; removed GND
- sheet SSD2 ports: added RelayGND; removed GND
- note added: "default is 5v processsor but dni resistors may be used to change to 3v3"

Commit message: progress on pcb
Connections:
- net at R35.1, U10.7 (B): now also J6.1; no longer J6.2
- net at R35.2, U10.8 (A): now also J6.2; no longer J6.1
- net at U10.5 (Y): now also J7.1; no longer J7.2
- net at U10.6 (Z): now also J7.2; no longer J7.1
Changed lines of the file:
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@@
 	(symbol
 		(lib_id "SamacSys_Parts:1935161")
-		(at 257.81 39.37 0)
-		(unit 1)
-		(exclude_from_sim no)
-		(in_bom yes)
-		(on_board yes)
-		(dnp no)
-		(fields_autoplaced yes)
+		(at 257.81 41.91 0)
+		(mirror x)
+		(unit 1)
+		(exclude_from_sim no)
+		(in_bom yes)
+		(on_board yes)
+		(dnp no)
 		(property "Reference" "J6"
-			(at 274.32 39.3699 0)
+			(at 274.32 41.9101 0)
 			(effects
 				(font
@@
 		)
 		(property "Value" "1935161"
-			(at 274.32 41.9099 0)
+			(at 274.32 39.3701 0)
 			(effects
 				(font
@@
 		)
 		(property "Footprint" "SamacSys_Parts:1935161"
+			(at 274.32 44.45 0)
+			(effects
+				(font
+					(size 1.27 1.27)
+				)
+				(justify left)
+				(hide yes)
+			)
+		)
+		(property "Datasheet" "https://www.mouser.com/ProductDetail/Phoenix-Contact/1935161?qs=W3wJikR1%252BS6eKzfFl8Rbew%3D%3D"
+			(at 274.32 41.91 0)
+			(effects
+				(font
+					(size 1.27 1.27)
+				)
+				(justify left)
+				(hide yes)
+			)
+		)
+		(property "Description" "Phoenix Contact COMBICON PT PCB Terminal Block, 2 Way/Pole, Screw Terminals, 26  14 AWG Through Hole, Nylon"
+			(at 257.81 41.91 0)
+			(effects
+				(font
+					(size 1.27 1.27)
+				)
+				(hide yes)
+			)
+		)
+		(property "Description_1" "Phoenix Contact COMBICON PT PCB Terminal Block, 2 Way/Pole, Screw Terminals, 26  14 AWG Through Hole, Nylon"
+			(at 274.32 39.37 0)
+			(effects
+				(font
+					(size 1.27 1.27)
+				)
+				(justify left)
+				(hide yes)
+			)
+		)
+		(property "Height" "11.55"
 			(at 274.32 36.83 0)
 			(effects
@@
 			)
 		)
-		(property "Datasheet" "https://www.mouser.com/ProductDetail/Phoenix-Contact/1935161?qs=W3wJikR1%252BS6eKzfFl8Rbew%3D%3D"
-			(at 274.32 39.37 0)
-			(effects
-				(font
-					(size 1.27 1.27)
-				)
-				(justify left)
-				(hide yes)
-			)
-		)
-		(property "Description" "Phoenix Contact COMBICON PT PCB Terminal Block, 2 Way/Pole, Screw Terminals, 26  14 AWG Through Hole, Nylon"
-			(at 257.81 39.37 0)
-			(effects
-				(font
-					(size 1.27 1.27)
-				)
-				(hide yes)
-			)
-		)
-		(property "Description_1" "Phoenix Contact COMBICON PT PCB Terminal Block, 2 Way/Pole, Screw Terminals, 26  14 AWG Through Hole, Nylon"
-			(at 274.32 41.91 0)
-			(effects
-				(font
-					(size 1.27 1.27)
-				)
-				(justify left)
-				(hide yes)
-			)
-		)
-		(property "Height" "11.55"
-			(at 274.32 44.45 0)
-			(effects
-				(font
-					(size 1.27 1.27)
-				)
-				(justify left)
-				(hide yes)
-			)
-		)
 		(property "Mouser Part Number" "651-1935161"
-			(at 274.32 46.99 0)
+			(at 274.32 34.29 0)
 			(effects
 				(font
@@
 		)
 		(property "Mouser Price/Stock" "https://www.mouser.co.uk/ProductDetail/Phoenix-Contact/1935161?qs=W3wJikR1%252BS6eKzfFl8Rbew%3D%3D"
-			(at 274.32 49.53 0)
+			(at 274.32 31.75 0)
 			(effects
 				(font
@@
 		)
 		(property "Manufacturer_Name" "Phoenix Contact"
-			(at 274.32 52.07 0)
+			(at 274.32 29.21 0)
 			(effects
 				(font
@@
 		)
 		(property "Manufacturer_Part_Number" "1935161"
-			(at 274.32 54.61 0)
+			(at 274.32 26.67 0)
 			(effects
 				(font
@@
 	(symbol
 		(lib_id "SamacSys_Parts:1935161")
-		(at 257.81 46.99 0)
-		(unit 1)
-		(exclude_from_sim no)
-		(in_bom yes)
-		(on_board yes)
-		(dnp no)
-		(fields_autoplaced yes)
+		(at 257.81 49.53 0)
+		(mirror x)
+		(unit 1)
+		(exclude_from_sim no)
+		(in_bom yes)
+		(on_board yes)
+		(dnp no)
 		(property "Reference" "J7"
-			(at 274.32 46.9899 0)
+			(at 274.32 49.5301 0)
 			(effects
 				(font
@@
 		)
 		(property "Value" "1935161"
-			(at 274.32 49.5299 0)
+			(at 274.32 46.9901 0)
 			(effects
 				(font
@@
 		)
 		(property "Footprint" "SamacSys_Parts:1935161"
+			(at 274.32 52.07 0)
+			(effects
+				(font
+					(size 1.27 1.27)
+				)
+				(justify left)
+				(hide yes)
+			)
+		)
+		(property "Datasheet" "https://www.mouser.com/ProductDetail/Phoenix-Contact/1935161?qs=W3wJikR1%252BS6eKzfFl8Rbew%3D%3D"
+			(at 274.32 49.53 0)
+			(effects
+				(font
+					(size 1.27 1.27)
+				)
+				(justify left)
+				(hide yes)
+			)
+		)
+		(property "Description" "Phoenix Contact COMBICON PT PCB Terminal Block, 2 Way/Pole, Screw Terminals, 26  14 AWG Through Hole, Nylon"
+			(at 257.81 49.53 0)
+			(effects
+				(font
+					(size 1.27 1.27)
+				)
+				(hide yes)
+			)
+		)
+		(property "Description_1" "Phoenix Contact COMBICON PT PCB Terminal Block, 2 Way/Pole, Screw Terminals, 26  14 AWG Through Hole, Nylon"
+			(at 274.32 46.99 0)
+			(effects
+				(font
+					(size 1.27 1.27)
+				)
+				(justify left)
+				(hide yes)
+			)
+		)
+		(property "Height" "11.55"
 			(at 274.32 44.45 0)
 			(effects
@@
 			)
 		)
-		(property "Datasheet" "https://www.mouser.com/ProductDetail/Phoenix-Contact/1935161?qs=W3wJikR1%252BS6eKzfFl8Rbew%3D%3D"
-			(at 274.32 46.99 0)
-			(effects
-				(font
-					(size 1.27 1.27)
-				)
-				(justify left)
-				(hide yes)
-			)
-		)
-		(property "Description" "Phoenix Contact COMBICON PT PCB Terminal Block, 2 Way/Pole, Screw Terminals, 26  14 AWG Through Hole, Nylon"
-			(at 257.81 46.99 0)
-			(effects
-				(font
-					(size 1.27 1.27)
-				)
-				(hide yes)
-			)
-		)
-		(property "Description_1" "Phoenix Contact COMBICON PT PCB Terminal Block, 2 Way/Pole, Screw Terminals, 26  14 AWG Through Hole, Nylon"
-			(at 274.32 49.53 0)
-			(effects
-				(font
-					(size 1.27 1.27)
-				)
-				(justify left)
-				(hide yes)
-			)
-		)
-		(property "Height" "11.55"
-			(at 274.32 52.07 0)
-			(effects
-				(font
-					(size 1.27 1.27)
-				)
-				(justify left)
-				(hide yes)
-			)
-		)
 		(property "Mouser Part Number" "651-1935161"
-			(at 274.32 54.61 0)
+			(at 274.32 41.91 0)
 			(effects
 				(font
@@
 		)
 		(property "Mouser Price/Stock" "https://www.mouser.co.uk/ProductDetail/Phoenix-Contact/1935161?qs=W3wJikR1%252BS6eKzfFl8Rbew%3D%3D"
-			(at 274.32 57.15 0)
+			(at 274.32 39.37 0)
 			(effects
 				(font
@@
 		)
 		(property "Manufacturer_Name" "Phoenix Contact"
-			(at 274.32 59.69 0)
+			(at 274.32 36.83 0)
 			(effects
 				(font
@@
 		)
 		(property "Manufacturer_Part_Number" "1935161"
-			(at 274.32 62.23 0)
-			(effects
-				(font
+			(at 274.32 34.29 0)
+			(effects
+				(font

Commit message: start switching to rp2040 and esp32
Parts:
- removed A2: Arduino_Nano_v3.x, Module:Arduino_Nano, symbol MCU_Module:Arduino_Nano_v3.x
- removed C11: 0.01uf, Capacitor_SMD:C_0402_1005Metric, symbol Device:C
- removed J6, J7: 1935161, SamacSys_Parts:1935161, symbol SamacSys_Parts:1935161
- removed R26, R29, R30, R31, R32: 0, Resistor_SMD:R_0805_2012Metric, symbol Device:R
- removed R33: 10k, Resistor_SMD:R_0402_1005Metric, symbol Device:R
- removed R35: 120, Resistor_SMD:R_0402_1005Metric, symbol Device:R
- removed SW2: SW_Push, Button_Switch_SMD:SW_Push_1P1T_NO_E-Switch_TL3301NxxxxxG, symbol Switch:SW_Push
- removed U10: MAX3490xSA, Package_SO:SOIC-8_3.9x4.9mm_P1.27mm, symbol Interface_UART:MAX3490xSA
- removed U8, U9: TXS0108EPW, Package_SO:TSSOP-20_4.4x6.5mm_P0.65mm, symbol Logic_LevelTranslator:TXS0108EPW
- added U18: ESP32-S3-DevKitC, PCM_Espressif:ESP32-S3-DevKitC, symbol PCM_Espressif:ESP32-S3-DevKitC
Connections:
- net thermoDrdy_3.3 is gone; now on net thermoDrdy: D14.2, D15.2, D16.2, D17.2, R21.1
- net thermoFault_3.3 is gone; now on net thermoFault: D10.2, D11.2, D12.2, D13.2, R19.1
- net 5V_Main: now also U18.21 (5V)
- net CLK: now also U18.18 (GPIO12/ADC2_CH1)
- net GND_Main: now also U18.22 (GND), U18.23 (GND), U18.24 (GND), U18.44 (GND)
- net MISO: now also U18.19 (GPIO13/ADC2_CH2)
- net MOSI: now also U18.17 (GPIO11/ADC2_CH0)
- new net: U18.1 (3V3), U18.2 (3V3)
- no-connect marks 0 -> 8
Other:
- note removed: "default is 5v processsor but dni resistors may be used to change to 3v3"
- note removed: "rs485"
- moved on the sheet: R19, R21, R34

Commit message: sch progress
Parts:
- removed D10, D11, D12, D13, D14, D15, D16, D17: SS16FP, SamacSys_Parts:SS12FP, symbol SamacSys_Parts:SS16FP
- added R35, R76, R77, R78: 10k, Resistor_SMD:R_0402_1005Metric, symbol Device:R
Connections:
- net thermoDrdy is gone; now on net thermoDrdy_0: R21.1
- net thermoFault is gone; now on net thermoFault_0: R19.1
- net 3.3V_Main: now also R20.2, R22.2, R23.2, R24.2, R25.2, R28.2, R34.2, R35.2, R76.2, R77.2, R78.2
- net 5V_Main: no longer R20.2, R22.2, R23.2, R24.2, R25.2, R28.2, R34.2
- net CS0: now also U18.20 (GPIO14/ADC2_CH3)
- net CS1: now also U18.10 (GPIO17/ADC2_CH6)
- net CS2: now also U18.11 (GPIO18/ADC2_CH7)
- net DataFromSafty: now also U18.27 (GPIO21)
- net DataToSafty: now also U18.32 (GPIO35)
- net Fault: now also U18.33 (GPIO36)
- net Relay1: now also U18.7 (GPIO7/ADC1_CH6)
- net Relay2: now also U18.12 (GPIO8/ADC1_CH7)
- net Relay3: now also U18.15 (GPIO9/ADC1_CH8)
- net thermoDrdy_1: now reaches U18.14 (GPIO46)
- net thermoDrdy_1: now also R76.1
- net Relay4: now reaches U18.16 (GPIO10/ADC1_CH9)
- net thermoFault_2: now reaches U18.28 (GPIO47)
- net thermoFault_2: now also R77.1
- net thermoDrdy_2: now reaches U18.29 (GPIO48)
- net thermoDrdy_2: now also R78.1
- net thermoFault_1: now reaches U18.30 (GPIO45)
- net thermoFault_1: now also R35.1
- net thermoFault_0: now reaches U18.34 (GPIO37)
- net thermoDrdy_0: now reaches U18.35 (GPIO38)
Other:
- sheet SSD renamed AuxRelay
- sheet SSD1 renamed Relay1
- sheet SSD2 renamed Relay2
- removed sheet Thermocouple
- added sheet Relay3 (SSD.kicad_sch)
- moved on the sheet: R19, R20, R21, R22, R23, R24, R25, R27, R28, R34, U18

Commit message: progress. still need to finish review
Parts:
- added R91, R92: 0, Resistor_SMD:R_0402_1005Metric, symbol Device:R
Connections:
- net 3.3V_Main: now also R91.2
- net 5V_Main: now also R92.2; no longer U18.21 (5V)
- net thermoDrdy_1: now also U18.6 (GPIO6/ADC1_CH5); no longer U18.14 (GPIO46)
- net thermoFault_1: now also U18.5 (GPIO5/ADC1_CH4); no longer U18.30 (GPIO45)
- net at U18.1 (3V3), U18.2 (3V3): now also R91.1
- new net: R92.1, U18.21 (5V)
- no-connect marks 8 -> 10
