File: MainControler.kicad_sch (KiCad schematic)
At the start: 17 parts, among them U18 ESP32-S3-DevKitC

Commit message: progress
Parts:
- removed R92: 0, Resistor_SMD:R_0402_1005Metric, symbol Device:R
- added C57: 0.1uf, Capacitor_SMD:C_0402_1005Metric, symbol Device:C
- R91: now fitted
Connections:
- net 3.3V_Main: now also C57.1
- net CS3: now also U18.27 (GPIO21)
- net DataFromSafty: now also U18.5 (GPIO5/ADC1_CH4); no longer U18.27 (GPIO21)
- net DataToSafty: now also U18.4 (GPIO4/ADC1_CH3); no longer U18.32 (GPIO35)
- net Fault: now also U18.6 (GPIO6/ADC1_CH5); no longer U18.33 (GPIO36)
- net GND_Main: now also C57.2
- net thermoDrdy_0: now also U18.31 (GPIO0); no longer U18.35 (GPIO38)
- net thermoDrdy_1: now also U18.41 (GPIO1/ADC1_CH0); no longer U18.6 (GPIO6/ADC1_CH5)
- net thermoDrdy_2: now also U18.40 (GPIO2/ADC1_CH1); no longer U18.29 (GPIO48)
- net thermoFault_0: now also U18.35 (GPIO38); no longer U18.34 (GPIO37)
- net thermoFault_1: now also U18.28 (GPIO47); no longer U18.5 (GPIO5/ADC1_CH4)
- net thermoFault_2: now also U18.29 (GPIO48); no longer U18.28 (GPIO47)
- no-connect marks 10 -> 14
Other:
- note added: "SCREEN IS CS3"
- moved on the sheet: R34

Commit message: sch looks prety good
Parts:
- removed R91: 0, Resistor_SMD:R_0402_1005Metric, symbol Device:R
- added C71, C72: 0.1uf, Capacitor_SMD:C_0402_1005Metric, symbol Device:C
- added J1: Conn_01x10_Pin, Connector_JST:JST_XH_B10B-XH-AM_1x10_P2.50mm_Vertical, symbol Connector:Conn_01x10_Pin
- added R26, R29: 2.2k, Resistor_SMD:R_0402_1005Metric, symbol Device:R
- added R30, R58, R61, R62: 10k, Resistor_SMD:R_0402_1005Metric, symbol Device:R
- added U7: SX1509, PCM_SparkFun-Semiconductor-Standard:QFN-28-1EP_4x4mm_P0.4mm_EP2.6x2.6mm, symbol PCM_SparkFun-IC-Special-Function:SX1509
Connections:
- net 3.3V_Main: now also U18.1 (3V3), U18.2 (3V3), C71.1, R26.2, R29.2, R58.2, R61.2, R62.2, U7.12 (VDDM), U7.18 (VCC2), U7.4 (VCC1)
- net CLK: now also J1.6 (Pin_6)
- net CS3: now also J1.5 (Pin_5)
- net MISO: now also J1.8 (Pin_8)
- net MOSI: now also J1.7 (Pin_7)
- net Relay1: now also U7.27 (I/O[0]); no longer U18.7 (GPIO7/ADC1_CH6)
- net Relay2: now also U7.28 (I/O[1]); no longer U18.12 (GPIO8/ADC1_CH7)
- net Relay3: now also U7.1 (I/O[2]); no longer U18.15 (GPIO9/ADC1_CH8)
- net Relay4: now also U7.2 (I/O[3]); no longer U18.16 (GPIO10/ADC1_CH9)
- net thermoDrdy_0: now also U7.13 (I/O[8]); no longer U18.31 (GPIO0)
- net thermoDrdy_1: now also U7.14 (I/O[9]); no longer U18.41 (GPIO1/ADC1_CH0)
- net thermoDrdy_2: now also U7.15 (I/O[10]); no longer U18.40 (GPIO2/ADC1_CH1)
- net GND_Main renamed GND
- net GND: now also C71.2, C72.2, J1.9 (Pin_9), R30.1, U7.10 (ADDR1), U7.17 (GND), U7.26 (ADDR0), U7.29 (GND), U7.3 (GND)
- new net 5V_Main: C72.1, J1.10 (Pin_10)
- new net IO_Expander_IRQ: R61.1, U18.7 (GPIO7/ADC1_CH6), U7.9 (~{INT})
- new net IO_Expander_RST: R62.1, U18.16 (GPIO10/ADC1_CH9), U7.23 (~{RESET})
- new net LCD_IORQ: J1.1 (Pin_1), R58.1, U7.21 (I/O[14])
- new net LCD_Reset: J1.4 (Pin_4), R30.2, U7.22 (I/O[15])
- new net SCL: J1.3 (Pin_3), R29.1, U18.15 (GPIO9/ADC1_CH8), U7.25 (SCL)
- new net SDA: J1.2 (Pin_2), R26.1, U18.12 (GPIO8/ADC1_CH7), U7.24 (SDA)
Other:
- note added: "BIGTREETECH TFT35 SPI V2.1 Touch Screen"
- note removed: "SCREEN IS CS3"
- moved on the sheet: C57, R19, R20, R21, R22, R23, R24, R25, R27, R28, R34, R35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
