File: Regulators.kicad_sch (KiCad schematic)
At the start: 20 parts, among them IC1 LT8631IFE#PBF, J10 1935161, U12 LM1117T-3.3

Commit message: progress. still need to finish review
Parts:
- removed U12: LM1117T-3.3, Package_TO_SOT_THT:TO-220-3_Vertical, symbol Regulator_Linear:LM1117T-3.3
- added U1: AP7361C-33E, Package_TO_SOT_SMD:SOT-223-3_TabPin2, symbol Regulator_Linear:AP7361C-33E
Connections:
- net 3.3V: now also U1.3 (VO)
- net 5V: now also U1.1 (VI)
- net PwrGnd: now also U1.2 (GND)
Other:
- note added: "set feedback for 5v!!!!!!!!!!!!!!"
