File: Regulators.kicad_sch (KiCad schematic)
At the start: 20 parts, among them IC1 LT8631IFE#PBF, J10 1935161, U1 AP7361C-33E

Commit message: progress
Parts:
- removed C22: 0.1uf, Capacitor_SMD:C_0402_1005Metric, symbol Device:C
- removed C24: 10uf 16v, Capacitor_SMD:C_0805_2012Metric, symbol Device:C
- removed L1: 15u (14.2u) 2A, Inductor_SMD:L_Chilisin_BMRF00101040, symbol Device:L
- removed U1: AP7361C-33E, Package_TO_SOT_SMD:SOT-223-3_TabPin2, symbol Regulator_Linear:AP7361C-33E
- added L3: 4.7uH 3.16A, WE-PD_7332/7345_PLASTIC_BASE54, symbol SamacSys_Parts:7447779004
- R47: value 422k -> 1M
- R48: value 47.5k -> 324k
Connections:
- net 5V is gone; now on net 3.3V: C17.1, C21.1, C23.2, IC1.12 (VOUT), R47.1
- net at C20.1, IC1.20 (SW): now also L3.1
- net at IC1.14 (IND): now also L3.2
Other:
- note removed: "set feedback for 5v!!!!!!!!!!!!!!"
- moved on the sheet: C16, R46
