File: SSD.kicad_sch (KiCad schematic)
At the start: 9 parts, among them J8 1935174, K1 EE2-12NUH, Q1 BSS138P,215

Commit message: progress
Parts:
- removed D26: SS16FP, SamacSys_Parts:SS12FP, symbol SamacSys_Parts:SS16FP
- added C7: 4.7pF, Capacitor_SMD:C_0402_1005Metric, symbol Device:C
- added D2: SMAJ24CA, Diode_SMD:D_SMA, symbol Diode:SMAJ24CA
- renumbered D18 to D1, J8 to J3, R36 to R33, R37 to R34, R82 to R35, R38 to R36
Connections:
- net RelayGND: now also C7.2, D2.1 (A1)
- net at D1.2, K1.12, Q1.3 (D)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: now also C7.1, D2.2 (A2)
