File: Thermocouple.kicad_sch (KiCad schematic)
At the start: 12 parts, among them J10 1935161, U10 MAX31856

Commit message: start adding switching pre-regulator
start isolating ground
Parts:
- added FB1, FB2: L, Inductor_SMD:L_0603_1608Metric, symbol Device:L
- renumbered C23 to C29, C24 to C30, C25 to C31, C26 to C32, C27 to C33, R32 to R37, R33 to R38, R34 to R39, R35 to R40, R36 to R41
Connections:
- net at R38.1, U10.2 (BIAS): now also FB2.2; no longer J10.1
- net at J10.2: now also FB1.1; no longer R37.1
- new net: FB2.1, J10.1
- new net: FB1.2, R37.1
Other:
- moved on the sheet: J10

Commit message: sch progress
Parts:
- removed C30, C32, C33: 0.1uf, Capacitor_SMD:C_0402_1005Metric, symbol Device:C
- removed C31: 0.01uf, Capacitor_SMD:C_0402_1005Metric, symbol Device:C
- removed R37, R38: 100, Resistor_SMD:R_0402_1005Metric, symbol Device:R
- added C26, C28, C29: 0.1uf, Capacitor_SMD:C_0402_1005Metric, symbol Device:C
- added C27: 0.01uf, Capacitor_SMD:C_0402_1005Metric, symbol Device:C
- added R44, R45: 120, Resistor_SMD:R_0402_1005Metric, symbol Device:R
- FB1, FB2: value L -> 74269244182; footprint Inductor_SMD:L_0603_1608Metric -> Inductor_SMD:L_0402_1005Metric_Pad0.77x0.64mm_HandSolder; MPN MMZ1608B121CTAH0 -> (none)
- renumbered C29 to C25, J10 to J11, R39 to R46, R40 to R47, R41 to R48, U10 to U13
Connections:
- net 3.3V_A: now also C28.1
- net 3.3V_D: now also C29.1
- net TC_AGND: now also C27.2, C28.2
- net TC_DGnd: now also C29.2
- net at FB2.2, U13.2 (BIAS): now also R45.2
- net at U13.3 (T-): now also C26.2, C27.1, R45.1
- net at FB1.2: now also R44.2
- net at C25.2, U13.4 (T+): now also C26.1, R44.1

Commit message: more sch updates
Parts:
- renumbered R44 to R49, R45 to R50, R46 to R51, R47 to R52, R48 to R53
Changed lines of the file:
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@@
 		(on_board yes)
 		(dnp no)
-		(property "Reference" "R48"
+		(property "Reference" "R53"
 			(at 190.754 78.74 90)
 			(effects
@@
 			(project "kiln"
 				(path "/e9c1836b-d16f-494a-819b-41549a786e18/307f7e78-c7c7-4c1f-bfd5-4e5fce95f524/4928fe5c-e6c8-45bf-90f3-0f12755b9f9e"
-					(reference "R76")
-					(unit 1)
-				)
-				(path "/e9c1836b-d16f-494a-819b-41549a786e18/307f7e78-c7c7-4c1f-bfd5-4e5fce95f524/88b1d8bc-9aca-411e-bb97-2183f44238e8"
+					(reference "R81")
+					(unit 1)
+				)
+				(path "/e9c1836b-d16f-494a-819b-41549a786e18/307f7e78-c7c7-4c1f-bfd5-4e5fce95f524/88b1d8bc-9aca-411e-bb97-2183f44238e8"
+					(reference "R58")
+					(unit 1)
+				)
+				(path "/e9c1836b-d16f-494a-819b-41549a786e18/307f7e78-c7c7-4c1f-bfd5-4e5fce95f524/bc013942-c6be-49fa-b321-e4929f62929c"
+					(reference "R63")
+					(unit 1)
+				)
+				(path "/e9c1836b-d16f-494a-819b-41549a786e18/307f7e78-c7c7-4c1f-bfd5-4e5fce95f524/e55a10d3-d364-4c02-8371-0e9595bd54af"
+					(reference "R72")
+					(unit 1)
+				)
+				(path "/e9c1836b-d16f-494a-819b-41549a786e18/9d216770-eb40-4527-939f-01f0f376c505/352ff89a-b0c5-441e-9692-8c7c78c5ff81"
 					(reference "R53")
-					(unit 1)
-				)
-				(path "/e9c1836b-d16f-494a-819b-41549a786e18/307f7e78-c7c7-4c1f-bfd5-4e5fce95f524/bc013942-c6be-49fa-b321-e4929f62929c"
-					(reference "R58")
-					(unit 1)
-				)
-				(path "/e9c1836b-d16f-494a-819b-41549a786e18/307f7e78-c7c7-4c1f-bfd5-4e5fce95f524/e55a10d3-d364-4c02-8371-0e9595bd54af"
-					(reference "R67")
-					(unit 1)
-				)
-				(path "/e9c1836b-d16f-494a-819b-41549a786e18/9d216770-eb40-4527-939f-01f0f376c505/352ff89a-b0c5-441e-9692-8c7c78c5ff81"
-					(reference "R48")
 					(unit 1)
 				)
@@
 		(on_board yes)
 		(dnp no)
-		(property "Reference" "R44"
+		(property "Reference" "R49"
 			(at 107.442 78.994 90)
 			(effects
@@
 			(project "kiln"
 				(path "/e9c1836b-d16f-494a-819b-41549a786e18/307f7e78-c7c7-4c1f-bfd5-4e5fce95f524/4928fe5c-e6c8-45bf-90f3-0f12755b9f9e"
-					(reference "R72")
-					(unit 1)
-				)
-				(path "/e9c1836b-d16f-494a-819b-41549a786e18/307f7e78-c7c7-4c1f-bfd5-4e5fce95f524/88b1d8bc-9aca-411e-bb97-2183f44238e8"
+					(reference "R77")
+					(unit 1)
+				)
+				(path "/e9c1836b-d16f-494a-819b-41549a786e18/307f7e78-c7c7-4c1f-bfd5-4e5fce95f524/88b1d8bc-9aca-411e-bb97-2183f44238e8"
+					(reference "R54")
+					(unit 1)
+				)
+				(path "/e9c1836b-d16f-494a-819b-41549a786e18/307f7e78-c7c7-4c1f-bfd5-4e5fce95f524/bc013942-c6be-49fa-b321-e4929f62929c"
+					(reference "R59")
+					(unit 1)
+				)
+				(path "/e9c1836b-d16f-494a-819b-41549a786e18/307f7e78-c7c7-4c1f-bfd5-4e5fce95f524/e55a10d3-d364-4c02-8371-0e9595bd54af"
+					(reference "R68")
+					(unit 1)
+				)
+				(path "/e9c1836b-d16f-494a-819b-41549a786e18/9d216770-eb40-4527-939f-01f0f376c505/352ff89a-b0c5-441e-9692-8c7c78c5ff81"
 					(reference "R49")
-					(unit 1)
-				)
-				(path "/e9c1836b-d16f-494a-819b-41549a786e18/307f7e78-c7c7-4c1f-bfd5-4e5fce95f524/bc013942-c6be-49fa-b321-e4929f62929c"
-					(reference "R54")
-					(unit 1)
-				)
-				(path "/e9c1836b-d16f-494a-819b-41549a786e18/307f7e78-c7c7-4c1f-bfd5-4e5fce95f524/e55a10d3-d364-4c02-8371-0e9595bd54af"
-					(reference "R63")
-					(unit 1)
-				)
-				(path "/e9c1836b-d16f-494a-819b-41549a786e18/9d216770-eb40-4527-939f-01f0f376c505/352ff89a-b0c5-441e-9692-8c7c78c5ff81"
-					(reference "R44")
 					(unit 1)
 				)
@@
 		(on_board yes)
 		(dnp no)
-		(property "Reference" "R47"
+		(property "Reference" "R52"
 			(at 185.674 78.74 90)
 			(effects
@@
 			(project "kiln"
 				(path "/e9c1836b-d16f-494a-819b-41549a786e18/307f7e78-c7c7-4c1f-bfd5-4e5fce95f524/4928fe5c-e6c8-45bf-90f3-0f12755b9f9e"
-					(reference "R75")
-					(unit 1)
-				)
-				(path "/e9c1836b-d16f-494a-819b-41549a786e18/307f7e78-c7c7-4c1f-bfd5-4e5fce95f524/88b1d8bc-9aca-411e-bb97-2183f44238e8"
+					(reference "R80")
+					(unit 1)
+				)
+				(path "/e9c1836b-d16f-494a-819b-41549a786e18/307f7e78-c7c7-4c1f-bfd5-4e5fce95f524/88b1d8bc-9aca-411e-bb97-2183f44238e8"
+					(reference "R57")
+					(unit 1)
+				)
+				(path "/e9c1836b-d16f-494a-819b-41549a786e18/307f7e78-c7c7-4c1f-bfd5-4e5fce95f524/bc013942-c6be-49fa-b321-e4929f62929c"
+					(reference "R62")
+					(unit 1)
+				)
+				(path "/e9c1836b-d16f-494a-819b-41549a786e18/307f7e78-c7c7-4c1f-bfd5-4e5fce95f524/e55a10d3-d364-4c02-8371-0e9595bd54af"
+					(reference "R71")
+					(unit 1)
+				)
+				(path "/e9c1836b-d16f-494a-819b-41549a786e18/9d216770-eb40-4527-939f-01f0f376c505/352ff89a-b0c5-441e-9692-8c7c78c5ff81"
 					(reference "R52")
-					(unit 1)
-				)
-				(path "/e9c1836b-d16f-494a-819b-41549a786e18/307f7e78-c7c7-4c1f-bfd5-4e5fce95f524/bc013942-c6be-49fa-b321-e4929f62929c"
-					(reference "R57")
-					(unit 1)
-				)
-				(path "/e9c1836b-d16f-494a-819b-41549a786e18/307f7e78-c7c7-4c1f-bfd5-4e5fce95f524/e55a10d3-d364-4c02-8371-0e9595bd54af"
-					(reference "R66")
-					(unit 1)
-				)
-				(path "/e9c1836b-d16f-494a-819b-41549a786e18/9d216770-eb40-4527-939f-01f0f376c505/352ff89a-b0c5-441e-9692-8c7c78c5ff81"
-					(reference "R47")
 					(unit 1)
 				)
@@
 		(on_board yes)
 		(dnp no)
-		(property "Reference" "R46"
+		(property "Reference" "R51"
 			(at 180.594 78.74 90)
 			(effects
@@
 			(project "kiln"
 				(path "/e9c1836b-d16f-494a-819b-41549a786e18/307f7e78-c7c7-4c1f-bfd5-4e5fce95f524/4928fe5c-e6c8-45bf-90f3-0f12755b9f9e"
-					(reference "R74")
-					(unit 1)
-				)
-				(path "/e9c1836b-d16f-494a-819b-41549a786e18/307f7e78-c7c7-4c1f-bfd5-4e5fce95f524/88b1d8bc-9aca-411e-bb97-2183f44238e8"
+					(reference "R79")
+					(unit 1)
+				)
+				(path "/e9c1836b-d16f-494a-819b-41549a786e18/307f7e78-c7c7-4c1f-bfd5-4e5fce95f524/88b1d8bc-9aca-411e-bb97-2183f44238e8"
+					(reference "R56")
+					(unit 1)
+				)
+				(path "/e9c1836b-d16f-494a-819b-41549a786e18/307f7e78-c7c7-4c1f-bfd5-4e5fce95f524/bc013942-c6be-49fa-b321-e4929f62929c"
+					(reference "R61")
+					(unit 1)
+				)
+				(path "/e9c1836b-d16f-494a-819b-41549a786e18/307f7e78-c7c7-4c1f-bfd5-4e5fce95f524/e55a10d3-d364-4c02-8371-0e9595bd54af"
+					(reference "R70")
+					(unit 1)
+				)
+				(path "/e9c1836b-d16f-494a-819b-41549a786e18/9d216770-eb40-4527-939f-01f0f376c505/352ff89a-b0c5-441e-9692-8c7c78c5ff81"
 					(reference "R51")
-					(unit 1)
-				)
-				(path "/e9c1836b-d16f-494a-819b-41549a786e18/307f7e78-c7c7-4c1f-bfd5-4e5fce95f524/bc013942-c6be-49fa-b321-e4929f62929c"
-					(reference "R56")
-					(unit 1)
-				)
-				(path "/e9c1836b-d16f-494a-819b-41549a786e18/307f7e78-c7c7-4c1f-bfd5-4e5fce95f524/e55a10d3-d364-4c02-8371-0e9595bd54af"
-					(reference "R65")
-					(unit 1)
-				)
-				(path "/e9c1836b-d16f-494a-819b-41549a786e18/9d216770-eb40-4527-939f-01f0f376c505/352ff89a-b0c5-441e-9692-8c7c78c5ff81"
-					(reference "R46")
 					(unit 1)
 				)
@@
 		(on_board yes)
 		(dnp no)
-		(property "Reference" "R45"
+		(property "Reference" "R50"
 			(at 107.442 89.154 90)
 			(effects
@@
 			(project "kiln"
 				(path "/e9c1836b-d16f-494a-819b-41549a786e18/307f7e78-c7c7-4c1f-bfd5-4e5fce95f524/4928fe5c-e6c8-45bf-90f3-0f12755b9f9e"
-					(reference "R73")
-					(unit 1)
-				)
-				(path "/e9c1836b-d16f-494a-819b-41549a786e18/307f7e78-c7c7-4c1f-bfd5-4e5fce95f524/88b1d8bc-9aca-411e-bb97-2183f44238e8"
+					(reference "R78")
+					(unit 1)
+				)
+				(path "/e9c1836b-d16f-494a-819b-41549a786e18/307f7e78-c7c7-4c1f-bfd5-4e5fce95f524/88b1d8bc-9aca-411e-bb97-2183f44238e8"
+					(reference "R55")
+					(unit 1)
+				)
+				(path "/e9c1836b-d16f-494a-819b-41549a786e18/307f7e78-c7c7-4c1f-bfd5-4e5fce95f524/bc013942-c6be-49fa-b321-e4929f62929c"
+					(reference "R60")
+					(unit 1)
+				)
+				(path "/e9c1836b-d16f-494a-819b-41549a786e18/307f7e78-c7c7-4c1f-bfd5-4e5fce95f524/e55a10d3-d364-4c02-8371-0e9595bd54af"
+					(reference "R69")
+					(unit 1)
+				)
+				(path "/e9c1836b-d16f-494a-819b-41549a786e18/9d216770-eb40-4527-939f-01f0f376c505/352ff89a-b0c5-441e-9692-8c7c78c5ff81"
 					(reference "R50")
 					(unit 1)
 				)
-				(path "/e9c1836b-d16f-494a-819b-41549a786e18/307f7e78-c7c7-4c1f-bfd5-4e5fce95f524/bc013942-c6be-49fa-b321-e4929f62929c"
-					(reference "R55")
-					(unit 1)
-				)
-				(path "/e9c1836b-d16f-494a-819b-41549a786e18/307f7e78-c7c7-4c1f-bfd5-4e5fce95f524/e55a10d3-d364-4c02-8371-0e9595bd54af"
-					(reference "R64")
-					(unit 1)
-				)
-				(path "/e9c1836b-d16f-494a-819b-41549a786e18/9d216770-eb40-4527-939f-01f0f376c505/352ff89a-b0c5-441e-9692-8c7c78c5ff81"
-					(reference "R45")
-					(unit 1)
-				)
