File: Thermocouple.kicad_sch (KiCad schematic)
At the start: 14 parts, among them J11 1935161, U13 MAX31856

Commit message: progress
Parts:
- removed R51, R52, R53: 10k, Resistor_SMD:R_0402_1005Metric, symbol Device:R
- added C59: 0.01uf, Capacitor_SMD:C_0402_1005Metric, symbol Device:C
- added R92: 2k, Resistor_SMD:R_0402_1005Metric, symbol Device:R
- R49, R50: value 120 -> 2k
Connections:
- net TC_AGND: now also C59.2
- net at FB2.2, R50.2: now also R92.2; no longer U13.2 (BIAS)
- new net: C59.1, R92.1, U13.2 (BIAS)
Other:
- moved on the sheet: C28, C29

Commit message: progress
Parts:
- renumbered C25 to C17, C26 to C18, C27 to C19, C59 to C20, C28 to C21, C29 to C22, J11 to J5, R49 to R48, R50 to R49, R92 to R50, U13 to U6
