File: Thermocouple.kicad_sch (KiCad schematic)
At the start: 13 parts, among them J5 1935161, U6 MAX31856

Commit message: sch check came back clean
Parts:
- FB1, FB2: value 74269244182 -> 1.8k
Changed lines of the file:
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@@
 			)
 		)
-		(property "Datasheet" "https://www.mouser.com/ProductDetail/KEMET/C0402C182J5RACTU?qs=DBJr%252BvBUjU6HgfnnR9R1kg%3D%3D"
+		(property "Datasheet" "https://www.mouser.com/en/ProductDetail/Murata-Electronics/GCM155R71H104KE02J?qs=hNud%2FORuBR1wlwGPFWBVDg%3D%3D"
 			(at 186.69 118.11 0)
 			(hide yes)
@@
 			)
 		)
-		(property "Value" "74269244182"
+		(property "Value" "1.8k"
 			(at 96.52 78.74 90)
 			(hide yes)
@@
 			)
 		)
-		(property "Datasheet" "https://www.mouser.com/ProductDetail/KEMET/C0402C182J5RACTU?qs=DBJr%252BvBUjU6HgfnnR9R1kg%3D%3D"
+		(property "Datasheet" "https://www.mouser.com/en/ProductDetail/Murata-Electronics/GCM155R71H104KE02J?qs=hNud%2FORuBR1wlwGPFWBVDg%3D%3D"
 			(at 115.57 86.36 0)
 			(hide yes)
@@
 			)
 		)
-		(property "Datasheet" "https://www.mouser.com/ProductDetail/KEMET/C0402C182J5RACTU?qs=DBJr%252BvBUjU6HgfnnR9R1kg%3D%3D"
+		(property "Datasheet" "https://www.mouser.com/en/ProductDetail/Murata-Electronics/GCM155R71H104KE02J?qs=hNud%2FORuBR1wlwGPFWBVDg%3D%3D"
 			(at 171.45 118.11 0)
 			(hide yes)
@@
 			)
 		)
-		(property "Value" "74269244182"
+		(property "Value" "1.8k"
 			(at 96.52 88.9 90)
 			(hide yes)

Commit message: pcb update
Parts:
- added C69, C73: 2.2uF, Capacitor_SMD:C_1206_3216Metric, symbol Device:C
- added D28: NUP2105L, Package_TO_SOT_SMD:SOT-23, symbol Power_Protection:NUP2105L
- added FB13, FB9: 1.8k, Inductor_SMD:L_0402_1005Metric_Pad0.77x0.64mm_HandSolder, symbol Device:L
Connections:
- net 3.3V_A: now also FB9.2; no longer C21.1, U6.5 (AVDD)
- net 3.3V_D: now also FB13.2; no longer C22.1, U6.8 (DVDD)
- net TC_AGND: now also C69.2, D28.3 (A)
- net TC_DGnd: now also C73.2
- net at FB1.2, R48.2: now also D28.1 (K)
- net at FB2.2, R49.2, R50.2: now also D28.2 (K)
- new net: C22.1, C73.1, FB13.1, U6.8 (DVDD)
- new net: C21.1, C69.1, FB9.1, U6.5 (AVDD)
Other:
- note removed: "PCC-SMP-K-R"
- note removed: "https://www.adafruit.com/product/3263?srsltid=AfmBOorLUUCO0d8wNJHWYgz-R17mwZTRphK52e8XEiY23RgYEyE77N2W"
- moved on the sheet: C21, C22, FB1, FB2, J5

Commit message: start adding seprate Thermocouple Board, fix some errors
Parts:
- C69, C73: Mouser Part Number Alt (none) -> https://www.mouser.com/en/ProductDetail/Samsung-Electro-Mec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; Mouser Part Number Alt 2 (none) -> https://www.mouser.com/en/ProductDetail/Murata-Electronics/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; Mouser Part Number Alt 3 (none) -> https://www.mouser.com/en/ProductDetail/Murata-Electronics/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; Mouser Part Number Alt 4 (none) -> https://www.mouser.com/en/ProductDetail/KEMET/C1206C225K5RA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
- D28: Mouser (none) -> https://www.mouser.com/en/ProductDetail/Diotec-Semiconducto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; Mouser Part Number Alt (none) -> https://www.mouser.com/en/ProductDetail/onsemi/NUP2105LT1G?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; Mouser Part Number Alt 2 (none) -> https://www.mouser.com/en/ProductDetail/onsemi/SZNUP2105LT1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; Mouser Part Number Alt 3 (none) -> https://www.mouser.com/en/ProductDetail/onsemi/SZNUP2105LT3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
- R48, R49, R50: value 2k -> 2.2k; Mouser Part Number Alt (none) -> https://www.mouser.com/en/ProductDetail/Bourns/CR0402-JW-22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; Mouser Part Number Alt 2 (none) -> https://www.mouser.com/en/ProductDetail/KOA-Speer/RK73B1ETT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
Changed lines of the file:
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@@
+			)
+		)
+		(property "Mouser Part Number Alt 3" "https://www.mouser.com/en/ProductDetail/onsemi/SZNUP2105LT3G?qs=PJJcWtbOkNXrvSZpB7E7mw%3D%3D"
+			(at 89.535 104.775 0)
+			(hide yes)
+			(show_name no)
+			(do_not_autoplace no)
+			(effects
+				(font
+					(size 1.27 1.27)
+				)
+			)
+		)
+		(property "Mouser Part Number Alt 2" "https://www.mouser.com/en/ProductDetail/onsemi/SZNUP2105LT1G?qs=PJJcWtbOkNWqqZbXH80dfQ%3D%3D"
+			(at 89.535 104.775 0)
+			(hide yes)
+			(show_name no)
+			(do_not_autoplace no)
+			(effects
+				(font
+					(size 1.27 1.27)
+				)
+			)
+		)
+		(property "Mouser Part Number Alt" "https://www.mouser.com/en/ProductDetail/onsemi/NUP2105LT1G?qs=ZXBb0xZ9WeDHmiHN%252BYKtYA%3D%3D"
+			(at 89.535 104.775 0)
+			(hide yes)
+			(show_name no)
+			(do_not_autoplace no)
+			(effects
+				(font
+					(size 1.27 1.27)
+				)
+			)
+		)
+		(property "Mouser" "https://www.mouser.com/en/ProductDetail/Diotec-Semiconductor/NUP2105L?qs=OlC7AqGiEDnwfsnn7%252BuLZg%3D%3D"
+			(at 89.535 104.775 0)
+			(hide yes)
+			(show_name no)
+			(do_not_autoplace no)
+			(effects
+				(font
+					(size 1.27 1.27)
+				)
 			)
 		)
@@
 			)
 		)
+		(property "Mouser Part Number Alt 4" "https://www.mouser.com/en/ProductDetail/KEMET/C1206C225K5RACAUTO7210?qs=%252BfJPIY6s7PlNVZKyV3SAGA%3D%3D"
+			(at 130.81 63.5 0)
+			(hide yes)
+			(show_name no)
+			(do_not_autoplace no)
+			(effects
+				(font
+					(size 1.27 1.27)
+				)
+			)
+		)
+		(property "Mouser Part Number Alt 3" "https://www.mouser.com/en/ProductDetail/Murata-Electronics/GCM31CR71H225KA55L?qs=aEuGZpxfbxXH69FledLqTA%3D%3D"
+			(at 130.81 63.5 0)
+			(hide yes)
+			(show_name no)
+			(do_not_autoplace no)
+			(effects
+				(font
+					(size 1.27 1.27)
+				)
+			)
+		)
+		(property "Mouser Part Number Alt 2" "https://www.mouser.com/en/ProductDetail/Murata-Electronics/GRT31CR71H225KE13L?qs=qkDYIeTQ%252BEkhrDhfEIGgfg%3D%3D"
+			(at 130.81 63.5 0)
+			(hide yes)
+			(show_name no)
+			(do_not_autoplace no)
+			(effects
+				(font
+					(size 1.27 1.27)
+				)
+			)
+		)
+		(property "Mouser Part Number Alt" "https://www.mouser.com/en/ProductDetail/Samsung-Electro-Mechanics/CL31B225KBHNFNE?qs=%252B6g0mu59x7Ixea%2FwRKCoRw%3D%3D"
+			(at 130.81 63.5 0)
+			(hide yes)
+			(show_name no)
+			(do_not_autoplace no)
+			(effects
+				(font
+					(size 1.27 1.27)
+				)
+			)
+		)
 		(property "Description" "Unpolarized capacitor"
 			(at 130.81 63.5 0)
@@
 			)
 		)
-		(property "Value" "2k"
+		(property "Value" "2.2k"
 			(at 109.474 81.28 90)
 			(show_name no)
@@
 			)
 		)
-		(property "Datasheet" "https://www.mouser.com/ProductDetail/Vishay-Beyschlag/MCS04020C1200FE000?qs=sGAEpiMZZMtlubZbdhIBIMAhWB6%252BRofmsfIIZouqAvg%3D"
+		(property "Datasheet" "https://www.mouser.com/en/ProductDetail/TE-Connectivity-Holsworthy/CRGCQ0402J2K2?qs=sGAEpiMZZMtG0KNrPCHnjW0BEZmmc%252BDpYMUb5aIRivWnzZusksZArA%3D%3D"
+			(at 109.22 81.28 0)
+			(hide yes)
+			(show_name no)
+			(do_not_autoplace no)
+			(effects
+				(font
+					(size 1.27 1.27)
+				)
+			)
+		)
+		(property "Mouser Part Number Alt 2" "https://www.mouser.com/en/ProductDetail/KOA-Speer/RK73B1ETTP222J?qs=sGAEpiMZZMtG0KNrPCHnjV5PF2HVMrQCyFb5Jr3rn%252Bc%3D"
+			(at 109.22 81.28 0)
+			(hide yes)
+			(show_name no)
+			(do_not_autoplace no)
+			(effects
+				(font
+					(size 1.27 1.27)
+				)
+			)
+		)
+		(property "Mouser Part Number Alt" "https://www.mouser.com/en/ProductDetail/Bourns/CR0402-JW-222GLF?qs=sGAEpiMZZMtG0KNrPCHnjfC2zYK6Lg3%2FUswrnEfVCX0%3D"
 			(at 109.22 81.28 0)
 			(hide yes)
@@
 			)
 		)
+		(property "Mouser Part Number Alt 4" "https://www.mouser.com/en/ProductDetail/KEMET/C1206C225K5RACAUTO7210?qs=%252BfJPIY6s7PlNVZKyV3SAGA%3D%3D"
+			(at 161.29 58.42 0)
+			(hide yes)
+			(show_name no)
+			(do_not_autoplace no)
+			(effects
+				(font
+					(size 1.27 1.27)
+				)
+			)
+		)
+		(property "Mouser Part Number Alt 3" "https://www.mouser.com/en/ProductDetail/Murata-Electronics/GCM31CR71H225KA55L?qs=aEuGZpxfbxXH69FledLqTA%3D%3D"
+			(at 161.29 58.42 0)
+			(hide yes)
+			(show_name no)
+			(do_not_autoplace no)
+			(effects
+				(font
+					(size 1.27 1.27)
+				)
+			)
+		)
+		(property "Mouser Part Number Alt 2" "https://www.mouser.com/en/ProductDetail/Murata-Electronics/GRT31CR71H225KE13L?qs=qkDYIeTQ%252BEkhrDhfEIGgfg%3D%3D"
+			(at 161.29 58.42 0)
+			(hide yes)
+			(show_name no)
+			(do_not_autoplace no)
+			(effects
+				(font
+					(size 1.27 1.27)
+				)
+			)
+		)
+		(property "Mouser Part Number Alt" "https://www.mouser.com/en/ProductDetail/Samsung-Electro-Mechanics/CL31B225KBHNFNE?qs=%252B6g0mu59x7Ixea%2FwRKCoRw%3D%3D"
+			(at 161.29 58.42 0)
+			(hide yes)
+			(show_name no)
+			(do_not_autoplace no)
+			(effects
+				(font
+					(size 1.27 1.27)
+				)
+			)
+		)
 		(property "Description" "Unpolarized capacitor"
 			(at 161.29 58.42 0)
@@
 			)
 		)
-		(property "Value" "2k"
+		(property "Value" "2.2k"
 			(at 112.014 115.57 90)
 			(show_name no)
@@
 			)
 		)
-		(property "Datasheet" "https://www.mouser.com/ProductDetail/Vishay-Beyschlag/MCS04020C1200FE000?qs=sGAEpiMZZMtlubZbdhIBIMAhWB6%252BRofmsfIIZouqAvg%3D"
+		(property "Datasheet" "https://www.mouser.com/en/ProductDetail/TE-Connectivity-Holsworthy/CRGCQ0402J2K2?qs=sGAEpiMZZMtG0KNrPCHnjW0BEZmmc%252BDpYMUb5aIRivWnzZusksZArA%3D%3D"
+			(at 111.76 115.57 0)
+			(hide yes)
+			(show_name no)
+			(do_not_autoplace no)
+			(effects
+				(font
+					(size 1.27 1.27)
+				)
+			)
+		)
+		(property "Mouser Part Number Alt 2" "https://www.mouser.com/en/ProductDetail/KOA-Speer/RK73B1ETTP222J?qs=sGAEpiMZZMtG0KNrPCHnjV5PF2HVMrQCyFb5Jr3rn%252Bc%3D"
+			(at 111.76 115.57 0)
+			(hide yes)
+			(show_name no)
+			(do_not_autoplace no)
+			(effects
+				(font
+					(size 1.27 1.27)
+				)
+			)
+		)
+		(property "Mouser Part Number Alt" "https://www.mouser.com/en/ProductDetail/Bourns/CR0402-JW-222GLF?qs=sGAEpiMZZMtG0KNrPCHnjfC2zYK6Lg3%2FUswrnEfVCX0%3D"
 			(at 111.76 115.57 0)
 			(hide yes)
@@
 			)
 		)
-		(property "Value" "2k"
+		(property "Value" "2.2k"
 			(at 109.474 91.44 90)
 			(show_name no)
@@
 			)
 		)
-		(property "Datasheet" "https://www.mouser.com/ProductDetail/Vishay-Beyschlag/MCS04020C1200FE000?qs=sGAEpiMZZMtlubZbdhIBIMAhWB6%252BRofmsfIIZouqAvg%3D"
+		(property "Datasheet" "https://www.mouser.com/en/ProductDetail/TE-Connectivity-Holsworthy/CRGCQ0402J2K2?qs=sGAEpiMZZMtG0KNrPCHnjW0BEZmmc%252BDpYMUb5aIRivWnzZusksZArA%3D%3D"
 			(at 109.22 91.44 0)
 			(hide yes)
+			(show_name no)
+			(do_not_autoplace no)
+			(effects
+				(font
+					(size 1.27 1.27)
+				)
+			)
+		)
+		(property "Mouser Part Number Alt 2" "https://www.mouser.com/en/ProductDetail/KOA-Speer/RK73B1ETTP222J?qs=sGAEpiMZZMtG0KNrPCHnjV5PF2HVMrQCyFb5Jr3rn%252Bc%3D"
+			(at 109.22 91.44 0)
+			(hide yes)
+			(show_name no)
+			(do_not_autoplace no)
+			(effects
+				(font
+					(size 1.27 1.27)
+				)
+			)
+		)
+		(property "Mouser Part Number Alt" "https://www.mouser.com/en/ProductDetail/Bourns/CR0402-JW-222GLF?qs=sGAEpiMZZMtG0KNrPCHnjfC2zYK6Lg3%2FUswrnEfVCX0%3D"
+			(at 109.22 91.44 0)
+			(hide yes)
