File: SaftyProcessor.kicad_sch (KiCad schematic)
At the start: 18 parts, among them J5 1935161, U4 TCMT1109, U5 TCMT1109, U6 TCMT1109

Commit message: progress
Parts:
- added C56: 2.2uF, Capacitor_SMD:C_1206_3216Metric, symbol Device:C
- added C58: 0.1uf, Capacitor_SMD:C_0402_1005Metric, symbol Device:C
Connections:
- net 3.3v_Safty: now also C58.1
- net GND_Safty: now also C56.2, C58.2
- net at A2.35 (ADC_VREF): now also C56.1
Other:
- sheet CurrentSense ports: added VCC; removed none
- sheet CurrentSense1 ports: added VCC; removed none
- sheet CurrentSense2 ports: added VCC; removed none
- moved on the sheet: R89, R90
