File: SaftyProcessor.kicad_sch (KiCad schematic)
At the start: 20 parts, among them J5 1935161, U4 TCMT1109, U5 TCMT1109, U6 TCMT1109

Commit message: sch looks prety good
Parts:
- R12, R17, R18: value 680 -> 390
Changed lines of the file:
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@@
 			)
 		)
-		(property "Value" "680"
+		(property "Value" "390"
 			(at 209.804 116.84 90)
 			(show_name no)
@@
 			)
 		)
-		(property "Value" "680"
+		(property "Value" "390"
 			(at 244.094 104.14 90)
 			(show_name no)
@@
 			)
 		)
-		(property "Value" "680"
+		(property "Value" "390"
 			(at 240.284 77.47 90)
 			(show_name no)

Commit message: progress
Parts:
- renumbered A2 to A1, C58 to C1, C56 to C2, C10 to C3, J5 to J1, R89 to R1, R16 to R10, R18 to R11, R17 to R12, R90 to R2, R11 to R3, R31 to R4, R32 to R5, R33 to R6, R12 to R7, R15 to R8, R14 to R9, U6 to U1, U4 to U2, U5 to U3

Commit message: add mouser sch tooling
Parts:
- A1: Mouser (none) -> https://www.mouser.com/en/ProductDetail/Raspberry-Pi/SC0915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
Changed lines of the file:
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@@
+			)
+		)
+		(property "Mouser" "https://www.mouser.com/en/ProductDetail/Raspberry-Pi/SC0915?qs=T%252BzbugeAwjgnLi4azxXVFA%3D%3D"
+			(at 149.86 119.38 0)
+			(hide yes)
+			(show_name no)
+			(do_not_autoplace no)
+			(effects
+				(font
+					(size 1.27 1.27)
+				)
 			)
 		)

Commit message: start adding seprate Thermocouple Board, fix some errors
Parts:
- C2: Mouser Part Number Alt (none) -> https://www.mouser.com/en/ProductDetail/Samsung-Electro-Mec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; Mouser Part Number Alt 2 (none) -> https://www.mouser.com/en/ProductDetail/Murata-Electronics/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; Mouser Part Number Alt 3 (none) -> https://www.mouser.com/en/ProductDetail/Murata-Electronics/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; Mouser Part Number Alt 4 (none) -> https://www.mouser.com/en/ProductDetail/KEMET/C1206C225K5RA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
Changed lines of the file:
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@@
+			)
+		)
+		(property "Mouser Part Number Alt 4" "https://www.mouser.com/en/ProductDetail/KEMET/C1206C225K5RACAUTO7210?qs=%252BfJPIY6s7PlNVZKyV3SAGA%3D%3D"
+			(at 191.77 82.55 0)
+			(hide yes)
+			(show_name no)
+			(do_not_autoplace no)
+			(effects
+				(font
+					(size 1.27 1.27)
+				)
+			)
+		)
+		(property "Mouser Part Number Alt 3" "https://www.mouser.com/en/ProductDetail/Murata-Electronics/GCM31CR71H225KA55L?qs=aEuGZpxfbxXH69FledLqTA%3D%3D"
+			(at 191.77 82.55 0)
+			(hide yes)
+			(show_name no)
+			(do_not_autoplace no)
+			(effects
+				(font
+					(size 1.27 1.27)
+				)
+			)
+		)
+		(property "Mouser Part Number Alt 2" "https://www.mouser.com/en/ProductDetail/Murata-Electronics/GRT31CR71H225KE13L?qs=qkDYIeTQ%252BEkhrDhfEIGgfg%3D%3D"
+			(at 191.77 82.55 0)
+			(hide yes)
+			(show_name no)
+			(do_not_autoplace no)
+			(effects
+				(font
+					(size 1.27 1.27)
+				)
+			)
+		)
+		(property "Mouser Part Number Alt" "https://www.mouser.com/en/ProductDetail/Samsung-Electro-Mechanics/CL31B225KBHNFNE?qs=%252B6g0mu59x7Ixea%2FwRKCoRw%3D%3D"
+			(at 191.77 82.55 0)
+			(hide yes)
+			(show_name no)
+			(do_not_autoplace no)
+			(effects
+				(font
+					(size 1.27 1.27)
+				)
 			)
 		)
