File: untitled.kicad_sch (KiCad schematic)
At the start: 20 parts, among them IC1 LT8631IFE#PBF, J10 1935161

Commit message: sch looks prety good
Parts:
- removed C1: 470uf 50v, CAPAE1360X1450N, symbol SamacSys_Parts:UCM1H471MNJ1MS
- removed C13, C18: 2.2uF, Capacitor_SMD:C_1206_3216Metric, symbol Device:C
- removed C16, C17, C20: 0.1uf, Capacitor_SMD:C_0402_1005Metric, symbol Device:C
- removed C21: 4.7pF, Capacitor_SMD:C_0402_1005Metric, symbol Device:C
- removed C23: 47uF 16V, Capacitor_SMD:C_1210_3225Metric, symbol Device:C
- removed D22: SMAJ24CA, Diode_SMD:D_SMA, symbol Diode:SMAJ24CA
- removed D3: LED, LED_SMD:LED_0402_1005Metric, symbol Device:LED
- removed IC1: LT8631IFE#PBF, SamacSys_Parts:SOP65P640X120-21N, symbol SamacSys_Parts:LT8631IFE#PBF
- removed J10: 1935161, SamacSys_Parts:1935161, symbol SamacSys_Parts:1935161
- removed L2: 4.7uH 3.16A, Inductor_SMD:L_7.3x7.3_H4.5, symbol Device:L
- removed R44: 75k, Resistor_SMD:R_0402_1005Metric, symbol Device:R
- removed R45: 10k, Resistor_SMD:R_0402_1005Metric, symbol Device:R
- removed R46: 8.66k, Resistor_SMD:R_0402_1005Metric, symbol Device:R
- removed R47: 475k 1%, Resistor_SMD:R_0402_1005Metric, symbol Device:R
- removed R48: 154k 1%, Resistor_SMD:R_0402_1005Metric, symbol Device:R
- removed R91: 2.2k, Resistor_SMD:R_0805_2012Metric, symbol Device:R
- added C71: 470u 35v, Capacitor_SMD:CP_Elec_10x14.3, symbol Device:C_Polarized
- added C72, C74: 2.2uF, Capacitor_SMD:C_1206_3216Metric, symbol Device:C
- added C73, C75, C78: 0.1uf, Capacitor_SMD:C_0402_1005Metric, symbol Device:C
- added C76: 4.7pF, Capacitor_SMD:C_0402_1005Metric, symbol Device:C
- added C77: 47uF 16V, Capacitor_SMD:C_1210_3225Metric, symbol Device:C
- added D39: SMAJ24CA, Diode_SMD:D_SMA, symbol Diode:SMAJ24CA
- added IC4: LT8631IFE#PBF, SamacSys_Parts:SOP65P640X120-21N, symbol SamacSys_Parts:LT8631IFE#PBF
- added J23: 1935161, SamacSys_Parts:1935161, symbol SamacSys_Parts:1935161
- added L6: 4.7uH 3.16A, WE-PD_7332/7345_PLASTIC_BASE54, symbol SamacSys_Parts:7447779004
- added R107: 75k, Resistor_SMD:R_0402_1005Metric, symbol Device:R
- added R109: 8.66k, Resistor_SMD:R_0402_1005Metric, symbol Device:R
- added R110: 475k 1%, Resistor_SMD:R_0402_1005Metric, symbol Device:R
- added R111: 154k 1%, Resistor_SMD:R_0402_1005Metric, symbol Device:R
- R108: value 2.2k -> 10k; footprint Resistor_SMD:R_0805_2012Metric -> Resistor_SMD:R_0402_1005Metric
Connections:
- net 12V: now also C71.1, C72.1, D39.2 (A2), IC4.1 (VIN), J23.2, R107.1
- net 3.3V: now also C76.1, C77.2, C78.1, IC4.12 (VOUT), R110.1
- net PwrGnd: now also R108.2, C71.2, C72.2, C73.2, C74.2, C77.1, C78.2, D39.1 (A1), IC4.13 (NC_3), IC4.15 (NC_4), IC4.21 (GND), IC4.6 (NC_1), IC4.7 (SYNC/MODE), IC4.9 (NC_2), J23.1, R109.2, R111.2
- net at R108.1: now also IC4.3 (EN/UV), R107.2
- new net: IC4.8 (RT), R109.1
- new net: C75.1, IC4.20 (SW), L6.1
- new net: IC4.14 (IND), L6.2
- new net: C76.2, IC4.11 (FB), R110.2, R111.1
- new net: C73.1, IC4.10 (TR/SS)
- new net: C74.1, IC4.16 (INTVCC)
- new net: C75.2, IC4.18 (BST)
