File: kiln.kicad_pcb (KiCad board)
At the start: 2 copper layers, 259 parts, among them IC1 LT8631IFE#PBF, IC2 LT8631IFE#PBF, IC3 LT8631IFE#PBF, J1 1935161, J10 1935174, J11 1935174, J12 1935161, J13 SJ2-35813B-SMT-TR, J14 1935161, J15 SJ2-35813B-SMT-TR, J16 1935161, J17 SJ2-35813B-SMT-TR, J18 1935161, J19 1935161, J2 Conn_01x10_Pin, J20 1935161, J21 1935161, J23 1935161, J24 1935161, J25 1935161, J3 1935174, J4 1935174, J5 1935161, J6 1935161, J7 1935161, J8 1935174, J9 1935161, K1 EE2-12NUH, K2 EE2-12NUH, K3 EE2-12NUH, K4 EE2-12NUH, K5 EE2-12NUH, Q1 BSS138P,215, Q2 BSS138P,215, Q3 BSS138P,215, Q4 BSS138P,215, Q5 BSS138P,215, U1 TCMT1109, U10 LMV321, U11 LMV321, U12 LMV321, U2 TCMT1109, U3 TCMT1109, U4 ESP32-S3-DevKitC, U5 SX1509, U6 MAX31856, U7 MAX31856, U8 MAX31856, U9 MAX31856

Commit message: progress
Parts:
- C20, C21, C22, C32, C33, C34, C39, C40, C41, C45, C46, C58, D14, D15, R50, R56, R63, R76, R77, R95, R96, U10: moved to B.Cu
- moved D24 130.8 mm to (150.3, 82.8), turned to 90 degrees
- moved J18 127.9 mm to (143.3, 87.8), turned to -90 degrees
- moved C53 122.3 mm to (160.8, 74.5)
- moved C54 122.3 mm to (159.7, 85.0)
- moved R92 122.3 mm to (153.9, 87.3)
- moved R93 122.3 mm to (153.9, 88.5)
- moved C55 122.3 mm to (153.9, 93.0)
- moved C56 122.3 mm to (164.9, 91.5)
- moved C57 122.3 mm to (164.9, 88.0)
- moved C58 122.3 mm to (162.1, 93.3)
- moved C59 122.3 mm to (163.4, 96.0)
- moved C60 122.3 mm to (163.4, 98.3)
- moved D25 122.3 mm to (153.9, 90.3)
- moved IC2 122.3 mm to (159.6, 90.2)
- moved L2 122.3 mm to (172.4, 90.8)
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Other:
- board text removed: "why is c12 diffrent from c64?"

Commit message: most of placement done
Parts:
- C1, C2, C4, C48, C49, C5, C51, C52, D18, D19, D22, D23, R1, R11, R12, R13, R14, R15, R16, R17, R19, R2, R20, R21, R23, R24, R25, R26, R27, R28, R29, R3, R30, R31, R32, R4, R5, R6, R7, R8, R82, R83, R88, R89, R9, U1, U11, U12, U2, U3: moved to B.Cu
- moved C43 400.0 mm to (162.9, 49.3)
- moved D10 400.0 mm to (164.4, 42.8)
- moved D11 400.0 mm to (164.4, 46.3)
- moved J11 400.0 mm to (165.4, 20.3)
- moved K5 400.0 mm to (163.9, 33.3)
- moved Q5 400.0 mm to (165.9, 50.4)
- moved R68 400.0 mm to (169.4, 51.3)
- moved R69 400.0 mm to (168.9, 49.3)
- moved R70 400.0 mm to (166.9, 35.8)
- moved R71 400.0 mm to (160.9, 35.8)
- moved C8 325.8 mm to (144.7, 49.3)
- moved D3 325.8 mm to (146.2, 42.8)
- moved D4 325.8 mm to (146.2, 46.3)
- moved J4 325.8 mm to (147.2, 20.3)
- moved K2 325.8 mm to (145.7, 33.3)
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
Commit message: update layout
Parts:
- moved C10 65.7 mm to (163.0, 106.5)
- moved C11 65.7 mm to (171.0, 112.2)
- moved C12 65.7 mm to (169.5, 101.2)
- moved C13 65.7 mm to (166.0, 101.2)
- moved C14 65.7 mm to (171.2, 104.0)
- moved C15 65.7 mm to (174.0, 102.8)
- moved C16 65.7 mm to (176.2, 102.8)
- moved C9 65.7 mm to (152.5, 105.3)
- moved D5 65.7 mm to (168.2, 112.2)
- moved L1 65.7 mm to (168.8, 93.8)
- moved R43 65.7 mm to (165.2, 112.2)
- moved R44 65.7 mm to (166.5, 112.2)
- moved R45 65.7 mm to (169.8, 112.2)
- moved R46 65.7 mm to (171.2, 105.2)
- moved R47 65.7 mm to (171.2, 106.5)
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Routing:
- net (no net): vias 0 -> 5
Other:
- board outline added: 203 x 116 mm
- copper layers 2 -> 4

Commit message: progress
Parts:
- moved C10 5.94 mm to (157.5, 104.2)
- moved C11 5.94 mm to (165.5, 110.0)
- moved C12 5.94 mm to (164.0, 99.0)
- moved C13 5.94 mm to (160.5, 99.0)
- moved C14 5.94 mm to (165.8, 101.8)
- moved C15 5.94 mm to (168.5, 100.5)
- moved C16 5.94 mm to (170.8, 100.5)
- moved C9 5.94 mm to (147.0, 103.1)
- moved D5 5.94 mm to (162.8, 110.0)
- moved IC1 5.94 mm to (162.7, 104.3)
- moved L1 5.94 mm to (163.2, 91.5)
- moved R41 5.94 mm to (160.9, 112.8)
- moved R42 5.94 mm to (164.2, 112.8)
- moved R43 5.94 mm to (159.8, 110.0)
- moved R44 5.94 mm to (161.0, 110.0)
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
Commit message: add netclasses
Parts:
- moved R42 61.9 mm to (113.7, 76.9), turned to -90 degrees
- moved R41 61.3 mm to (113.7, 73.6), turned to -90 degrees
- moved C11 58.5 mm to (116.4, 78.2), turned to 180 degrees
- moved R45 58.1 mm to (116.4, 77.0), turned to 180 degrees
- moved D5 57.8 mm to (116.4, 75.5), turned to 180 degrees
- moved R44 57.5 mm to (116.4, 73.7), turned to 180 degrees
- moved R43 57.3 mm to (116.4, 72.5), turned to 0 degrees
- moved R47 50.6 mm to (122.2, 78.5), turned to 90 degrees
- moved IC1 49.9 mm to (122.1, 75.4), turned to 0 degrees
- moved C9 49.4 mm to (123.3, 59.7), turned to 0 degrees
- moved C10 49.0 mm to (122.2, 70.2), turned to 0 degrees
- moved R46 48.9 mm to (123.4, 78.5), turned to -90 degrees
- moved C16 48.0 mm to (125.9, 83.5), turned to 180 degrees
- moved C14 47.2 mm to (124.7, 78.5), turned to -90 degrees
- moved C15 46.8 mm to (125.9, 81.2), turned to 0 degrees
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
Commit message: routing almost done
Parts:
- moved J10 101.4 mm to (58.4, 79.4), turned to -90 degrees
- moved K4 83.5 mm to (71.8, 80.9), turned to -90 degrees
- moved R66 82.4 mm to (74.3, 77.9), turned to 180 degrees
- moved R67 78.4 mm to (74.3, 83.9), turned to 180 degrees
- moved D8 72.1 mm to (81.3, 80.4), turned to -90 degrees
- moved R65 68.4 mm to (87.8, 75.9), turned to 0 degrees
- moved D9 67.9 mm to (84.8, 80.4), turned to -90 degrees
- moved R64 66.8 mm to (89.8, 75.4), turned to 90 degrees
- moved Q4 64.6 mm to (88.8, 78.9), turned to -90 degrees
- moved C42 63.2 mm to (87.8, 81.9), turned to 90 degrees
- moved C3 22.4 mm to (65.5, 60.8)
- moved J1 22.4 mm to (59.5, 59.8)
- moved R10 22.4 mm to (65.5, 63.3)
- moved C56 8.59 mm to (155.8, 95.4)
- moved IC2 8.45 mm to (154.6, 101.8)
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Routing:
- net GND_Main: track 0.00 -> 182.1 mm, vias 0 -> 66
- net 12V_Main: track 0.00 -> 138.9 mm, vias 0 -> 13
- net GND_Safty: track 0.00 -> 117.8 mm, vias 0 -> 23
- net /MainControler/Relay1: track 0.00 -> 96.3 mm, vias 0 -> 4
- net /MainControler/MISO: track 0.00 -> 93.3 mm, vias 0 -> 4
- net /MainControler/MOSI: track 0.00 -> 93.2 mm, vias 0 -> 8
- net /MainControler/thermoFault_0: track 0.00 -> 91.3 mm, vias 0 -> 4
- net /MainControler/CLK: track 0.00 -> 90.3 mm
- net /MainControler/Relay2: track 0.00 -> 86.7 mm, vias 0 -> 4
- net /MainControler/CS1: track 0.00 -> 85.2 mm, vias 0 -> 2
- net /MainControler/Relay3: track 0.00 -> 84.8 mm, vias 0 -> 6
- net /MainControler/Relay4: track 0.00 -> 75.8 mm, vias 0 -> 4
- net /MainControler/CS0: track 0.00 -> 69.9 mm, vias 0 -> 2
- net /MainControler/SDA: track 0.00 -> 67.8 mm, vias 0 -> 8
- net /MainControler/LCD_IORQ: track 0.00 -> 66.7 mm, vias 0 -> 5
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- added copper zone on In2.Cu, net 12V_Main
- added copper zone on In2.Cu, net 3.3V_Main
- added copper zone on In2.Cu, net 3.3v_Safty
- added copper zone on B.Cu, net GND_Main
- added copper zone on F.Cu, net GND_Main
- added copper zone on In1.Cu, net GND_Main
- added copper zone on B.Cu, net GND_Safty
- added copper zone on F.Cu, net GND_Safty
- added copper zone on In1.Cu, net GND_Safty
