File: kiln.kicad_pcb (KiCad board)
At the start: 4 copper layers, 203 x 116 mm, 259 parts, among them IC1 LT8631IFE#PBF, IC2 LT8631IFE#PBF, IC3 LT8631IFE#PBF, J1 1935161, J10 1935174, J11 1935174, J12 1935161, J13 SJ2-35813B-SMT-TR, J14 1935161, J15 SJ2-35813B-SMT-TR, J16 1935161, J17 SJ2-35813B-SMT-TR, J18 1935161, J19 1935161, J2 Conn_01x10_Pin, J20 1935161, J21 1935161, J23 1935161, J24 1935161, J25 1935161, J3 1935174, J4 1935174, J5 1935161, J6 1935161, J7 1935161, J8 1935174, J9 1935161, K1 EE2-12NUH, K2 EE2-12NUH, K3 EE2-12NUH, K4 EE2-12NUH, K5 EE2-12NUH, Q1 BSS138P,215, Q2 BSS138P,215, Q3 BSS138P,215, Q4 BSS138P,215, Q5 BSS138P,215, U1 TCMT1109, U10 LMV321, U11 LMV321, U12 LMV321, U2 TCMT1109, U3 TCMT1109, U4 ESP32-S3-DevKitC, U5 SX1509, U6 MAX31856, U7 MAX31856, U8 MAX31856, U9 MAX31856

Commit message: progress
Parts:
- C53, C61, C9: value 470uf 50v -> 470uf
- FB1, FB2, FB3, FB4, FB5, FB6, FB7, FB8: value 74269244182 -> 1.8k
- R47: value 90.7k 1% -> 90.9k 1%
- moved R91 14.4 mm to (170.4, 108.4)
- moved C55 14.3 mm to (171.4, 104.8)
- moved C57 14.3 mm to (166.4, 93.8)
- moved C58 14.3 mm to (171.7, 96.6)
- moved C59 14.3 mm to (174.4, 95.3)
- moved C60 14.3 mm to (176.7, 95.3)
- moved D25 14.3 mm to (168.7, 104.8)
- moved L2 14.3 mm to (169.2, 86.3)
- moved R90 14.3 mm to (166.8, 107.6)
- moved R94 14.3 mm to (170.2, 104.8)
- moved R95 14.3 mm to (171.7, 97.8)
- moved R96 14.3 mm to (171.7, 99.1)
- moved C53 14.3 mm to (152.9, 97.9)
- moved C54 14.3 mm to (163.4, 99.0)
- moved C56 14.3 mm to (169.8, 92.8)
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Routing:
- net /MainControler/DataToSafty: track 0.00 -> 128.1 mm, vias 0 -> 3
- net /MainControler/DataFromSafty: track 0.00 -> 126.6 mm, vias 0 -> 3
- net /MainControler/Fault: track 0.00 -> 121.7 mm, vias 0 -> 2
- net GND_Safty: track 117.8 -> 228.7 mm, vias 23 -> 109
- net 5V_Main: track 19.1 -> 107.2 mm, vias 2 -> 4
- net /MainRegulator/PGoodMain: track 5.90 -> 89.1 mm, vias 0 -> 4
- net /MainControler/thermoFault_1: track 2.63 -> 61.2 mm, vias 0 -> 2
- net 12v_Safty: track 60.6 -> 118.3 mm, vias 5 -> 16
- net /SaftyProcessor/saftyRelay: track 0.00 -> 48.2 mm
- net /MainControler/thermoFault_2: track 2.62 -> 44.8 mm, vias 0 -> 1
- net GND_Main: track 182.1 -> 223.6 mm, vias 66 -> 251
- net /SaftyProcessor/estop: track 32.4 -> 73.5 mm
- net 12V_Main: track 138.9 -> 172.0 mm, vias 13 -> 19
- net 3.3V_Main: track 47.4 -> 59.3 mm, vias 26 -> 32
- net Net-(IC1-SW): track 11.1 -> 16.8 mm, vias 0 -> 2
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- added copper zone on B.Cu, net 12v_Safty
- added copper zone on F.Cu, net 12v_Safty
- added copper zone on In1.Cu, net 12v_Safty

Commit message: pcb update
Parts:
- added C69: 2.2uF, Capacitor_SMD:C_1206_3216Metric, B.Cu at (71.3, 128.0)
- added C70: 2.2uF, Capacitor_SMD:C_1206_3216Metric, B.Cu at (145.9, 126.2)
- added C71: 2.2uF, Capacitor_SMD:C_1206_3216Metric, B.Cu at (161.9, 130.3)
- added C72: 2.2uF, Capacitor_SMD:C_1206_3216Metric, B.Cu at (174.6, 131.1)
- added C73: 2.2uF, Capacitor_SMD:C_1206_3216Metric, B.Cu at (66.0, 125.9)
- added C75: 2.2uF, Capacitor_SMD:C_1206_3216Metric, B.Cu at (138.7, 127.0)
- added C77: 2.2uF, Capacitor_SMD:C_1206_3216Metric, B.Cu at (152.3, 127.3)
- added C79: 2.2uF, Capacitor_SMD:C_1206_3216Metric, B.Cu at (166.7, 127.5)
- added D28: NUP2105L, Package_TO_SOT_SMD:SOT-23, B.Cu at (67.4, 138.5)
- added D29: NUP2105L, Package_TO_SOT_SMD:SOT-23, B.Cu at (141.6, 138.1)
- added D30: NUP2105L, Package_TO_SOT_SMD:SOT-23, B.Cu at (155.8, 138.1)
- added D31: NUP2105L, Package_TO_SOT_SMD:SOT-23, B.Cu at (170.1, 138.4)
- added FB10: 1.8k, Inductor_SMD:L_0402_1005Metric_Pad0.77x0.64mm_HandSolder, B.Cu at (143.9, 128.3)
- added FB11: 1.8k, Inductor_SMD:L_0402_1005Metric_Pad0.77x0.64mm_HandSolder, B.Cu at (158.8, 128.6)
- added FB12: 1.8k, Inductor_SMD:L_0402_1005Metric_Pad0.77x0.64mm_HandSolder, B.Cu at (172.6, 129.0)
- added FB13: 1.8k, Inductor_SMD:L_0402_1005Metric_Pad0.77x0.64mm_HandSolder, B.Cu at (67.8, 127.3)
- added FB14: 1.8k, Inductor_SMD:L_0402_1005Metric_Pad0.77x0.64mm_HandSolder, B.Cu at (142.1, 127.3)
- added FB15: 1.8k, Inductor_SMD:L_0402_1005Metric_Pad0.77x0.64mm_HandSolder, B.Cu at (157.4, 127.8)
- added FB16: 1.8k, Inductor_SMD:L_0402_1005Metric_Pad0.77x0.64mm_HandSolder, B.Cu at (171.5, 127.5)
- added FB9: 1.8k, Inductor_SMD:L_0402_1005Metric_Pad0.77x0.64mm_HandSolder, B.Cu at (68.8, 128.2)
- added R104: 390, Resistor_SMD:R_0402_1005Metric, F.Cu at (238.9, 134.5)
- added R105: 390, Resistor_SMD:R_0402_1005Metric, F.Cu at (217.2, 131.7)
- added R106: 2.2k, Resistor_SMD:R_0402_1005Metric, F.Cu at (229.4, 131.7)
- added U13: TCMT1109, Package_SO:SOP-4_4.4x2.6mm_P1.27mm, F.Cu at (233.0, 134.4)
- added U14: TCMT1109, Package_SO:SOP-4_4.4x2.6mm_P1.27mm, F.Cu at (220.9, 134.5)
Connections:
- C21 pad 1: 3.3v_Safty -> Net-(U6-AVDD)
- C22 pad 1: 3.3v_Safty -> Net-(U6-DVDD)
- C27 pad 1: 3.3V_Main -> Net-(U7-AVDD)
- C28 pad 1: 3.3V_Main -> Net-(U7-DVDD)
- C33 pad 1: 3.3V_Main -> Net-(U8-AVDD)
- C34 pad 1: 3.3V_Main -> Net-(U8-DVDD)
- C40 pad 1: 3.3V_Main -> Net-(U9-AVDD)
- C41 pad 1: 3.3V_Main -> Net-(U9-DVDD)
- D12 pad 1: Net-(D12-A) -> GND_Safty
- D13 pad 1: Net-(D12-A) -> GND_Safty
- D16 pad 1: Net-(D16-A) -> GND_Safty
- D17 pad 1: Net-(D16-A) -> GND_Safty
- D20 pad 1: Net-(D20-A) -> GND_Safty
- D21 pad 1: Net-(D20-A) -> GND_Safty
- J20 pad 1: /MainControler/IO_4 -> /MainControler/IO_3
- J20 pad 2: GND_Main -> /MainControler/IO_4
- J24 pad 1: GND_Main -> Net-(J24-Pad1)
- J24 pad 2: /MainControler/IO_1 -> Net-(J24-Pad2)
- J25 pad 1: /MainControler/IO_2 -> Net-(J25-Pad1)
- J25 pad 2: /MainControler/IO_3 -> Net-(J25-Pad2)
- U6 pad 5: 3.3v_Safty -> Net-(U6-AVDD)
- U6 pad 8: 3.3v_Safty -> Net-(U6-DVDD)
- U7 pad 5: 3.3V_Main -> Net-(U7-AVDD)
- U7 pad 8: 3.3V_Main -> Net-(U7-DVDD)
- U8 pad 5: 3.3V_Main -> Net-(U8-AVDD)
- U8 pad 8: 3.3V_Main -> Net-(U8-DVDD)
- U9 pad 5: 3.3V_Main -> Net-(U9-AVDD)
- U9 pad 8: 3.3V_Main -> Net-(U9-DVDD)
Routing:
- net GND_Main: track 223.6 -> 246.2 mm, vias 251 -> 262
- net Net-(J24-Pad1): track 0.00 -> 17.4 mm
- net Net-(J25-Pad1): track 0.00 -> 11.6 mm
- net GND_Safty: track 228.7 -> 240.2 mm, vias 109 -> 111
- net Net-(J24-Pad2): track 0.00 -> 10.3 mm
- net Net-(U6-DVDD): track 0.00 -> 10.2 mm, vias 0 -> 1
- net Net-(U7-DVDD): track 0.00 -> 10.1 mm, vias 0 -> 1
- net Net-(U9-DVDD): track 0.00 -> 9.65 mm, vias 0 -> 1
- net Net-(U8-DVDD): track 0.00 -> 9.17 mm, vias 0 -> 1
- net Net-(J25-Pad2): track 0.00 -> 7.12 mm
- net Net-(U7-AVDD): track 0.00 -> 6.69 mm, vias 0 -> 1
- net Net-(U8-AVDD): track 0.00 -> 6.37 mm, vias 0 -> 1
- net /MainControler/IO_1: track 49.2 -> 55.1 mm
- net 3.3v_Safty: track 37.5 -> 31.9 mm
- net Net-(U9-AVDD): track 0.00 -> 5.51 mm, vias 0 -> 1
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