File: CurrentSense.kicad_sch (KiCad schematic)
At the start: 10 parts, among them J2 1935161, J4 SJ2-35813B-SMT-TR

Commit message: progress
Parts:
- removed C7: 10uf 16v, Capacitor_SMD:C_0805_2012Metric, symbol Device:C
- removed D3, D4, D7, D8: SS16FP, SamacSys_Parts:SS12FP, symbol SamacSys_Parts:SS16FP
- removed J4: SJ2-35813B-SMT-TR, SamacSys_Parts:SJ235813BSMTTR, symbol SamacSys_Parts:SJ2-35813B-SMT-TR
- removed R2: 100R 1W, Resistor_SMD:R_2512_6332Metric, symbol Device:R
- removed R4: 1k, Resistor_SMD:R_0402_1005Metric, symbol Device:R
- removed R6: 47.5k, Resistor_SMD:R_0402_1005Metric, symbol Device:R
- added C50: 0.1uf, Capacitor_SMD:C_0402_1005Metric, symbol Device:C
- added C53: 4.7pF, Capacitor_SMD:C_0402_1005Metric, symbol Device:C
- added C8: 10uf 16v, Capacitor_SMD:C_0805_2012Metric, symbol Device:C
- added D1, D16: BZX84C3V3LT1G, Package_TO_SOT_SMD:SOT-23, symbol Diode:BZX84Cxx
- added D12, D9: SS16FP, SamacSys_Parts:SS12FP, symbol SamacSys_Parts:SS16FP
- added J20: SJ2-35813B-SMT-TR, SamacSys_Parts:SJ235813BSMTTR, symbol SamacSys_Parts:SJ2-35813B-SMT-TR
- added R10, R7, R98: 47k, Resistor_SMD:R_0402_1005Metric, symbol Device:R
- added R101: 1M, Resistor_SMD:R_0402_1005Metric, symbol Device:R
- added R104: 100R 1W, Resistor_SMD:R_2512_6332Metric, symbol Device:R
- added U1: LMV321, Package_TO_SOT_SMD:SOT-353_SC-70-5, symbol Amplifier_Operational:LMV321
Connections:
- net Gnd: now also J2.1, C50.2, C8.2, D12.2, J20.1 (SLEEVE), R10.1, R101.2, R104.2, U1.2 (V-)
- net Vout: now also C8.1, D9.1, R101.1, R98.2
- net at J2.2: now also J20.2 (TIP), R104.1, R7.1
- new net: D1.1 (A), D16.1 (A)
- new net: C53.2, D16.3 (K), R10.2, R98.1, U1.3 (-)
- new net: C53.1, D1.3 (K), D12.1, R7.2, U1.1 (+)
- new net: D9.2, U1.4
- new net VCC: C50.1, U1.5 (V+)
- no-connect marks 2 -> 0

Commit message: sch looks prety good
Parts:
- added R13: 475k, Resistor_SMD:R_0402_1005Metric, symbol Device:R
- J2: now not fitted
Connections:
- net Gnd: now also J20.3 (RING), R13.1
- net at J2.2, J20.2 (TIP), R104.1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: now also R13.2
- no-connect marks 0 -> 1
Other:
- moved on the sheet: J20, R104

Commit message: progress
Parts:
- renumbered C53 to C44, C50 to C45, C8 to C46, D1 to D12, D16 to D13, D12 to D14, D9 to D15, J2 to J12, J20 to J13, R104 to R72, R13 to R73, R7 to R74, R10 to R75, R98 to R76, R101 to R77, U1 to U10

Commit message: progress
Parts:
- D12, D13: now fitted
Changed lines of the file:
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@@
 		(on_board yes)
 		(in_pos_files yes)
-		(dnp yes)
+		(dnp no)
 		(fields_autoplaced yes)
 		(property "Reference" "D13"
@@
 		(on_board yes)
 		(in_pos_files yes)
-		(dnp yes)
+		(dnp no)
 		(fields_autoplaced yes)
 		(property "Reference" "D12"

Commit message: pcb update
Connections:
- net Gnd: now also D12.1 (A), D13.1 (A)
Changed lines of the file:
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@@
+		(color 0 0 0 0)
+	)
+	(junction
+		(at 134.62 88.9)
+		(diameter 0)
 		(color 0 0 0 0)
 	)
@@
 	(wire
 		(pts
+			(xy 130.81 88.9) (xy 134.62 88.9)
+		)
+		(stroke
+			(width 0)
+			(type default)
+		)
+	)
+	(wire
+		(pts
 			(xy 220.98 104.14) (xy 220.98 106.68)
 		)
@@
 		(pts
 			(xy 226.06 93.98) (xy 232.41 93.98)
+		)
+		(stroke
+			(width 0)
+			(type default)
+		)
+	)
+	(wire
+		(pts
+			(xy 130.81 101.6) (xy 130.81 88.9)
 		)
 		(stroke
@@
 		)
 	)
+	(hierarchical_label "Gnd"
+		(shape passive)
+		(at 130.81 101.6 270)
+		(effects
+			(font
+				(size 1.27 1.27)
+			)
+			(justify right)
+		)
+	)
