File: 5V_Regulator.kicad_sch (KiCad schematic)
At the start: 20 parts, among them IC1 LT8631IFE#PBF, J10 1935161

Commit message: sch looks prety good
Parts:
- removed C1: 470uf 50v, CAPAE1360X1450N, symbol SamacSys_Parts:UCM1H471MNJ1MS
- removed C13, C18: 2.2uF, Capacitor_SMD:C_1206_3216Metric, symbol Device:C
- removed C16, C17, C20: 0.1uf, Capacitor_SMD:C_0402_1005Metric, symbol Device:C
- removed C21: 4.7pF, Capacitor_SMD:C_0402_1005Metric, symbol Device:C
- removed C23: 47uF 16V, Capacitor_SMD:C_1210_3225Metric, symbol Device:C
- removed D22: SMAJ24CA, Diode_SMD:D_SMA, symbol Diode:SMAJ24CA
- removed D3: LED, LED_SMD:LED_0402_1005Metric, symbol Device:LED
- removed IC1: LT8631IFE#PBF, SamacSys_Parts:SOP65P640X120-21N, symbol SamacSys_Parts:LT8631IFE#PBF
- removed J10: 1935161, SamacSys_Parts:1935161, symbol SamacSys_Parts:1935161
- removed L2: 4.7uH 3.16A, Inductor_SMD:L_7.3x7.3_H4.5, symbol Device:L
- removed R108, R91: 2.2k, Resistor_SMD:R_0805_2012Metric, symbol Device:R
- removed R44: 75k, Resistor_SMD:R_0402_1005Metric, symbol Device:R
- removed R45: 10k, Resistor_SMD:R_0402_1005Metric, symbol Device:R
- removed R46: 8.66k, Resistor_SMD:R_0402_1005Metric, symbol Device:R
- removed R47: 475k 1%, Resistor_SMD:R_0402_1005Metric, symbol Device:R
- removed R48: 154k 1%, Resistor_SMD:R_0402_1005Metric, symbol Device:R
- added C3: 470uf 50v, CAPAE1360X1450N, symbol SamacSys_Parts:UCM1H471MNJ1MS
- added C64, C66: 2.2uF, Capacitor_SMD:C_1206_3216Metric, symbol Device:C
- added C65, C67, C70: 0.1uf, Capacitor_SMD:C_0402_1005Metric, symbol Device:C
- added C68: 4.7pF, Capacitor_SMD:C_0402_1005Metric, symbol Device:C
- added C69: 47uF 16V, Capacitor_SMD:C_1210_3225Metric, symbol Device:C
- added D5: LED, LED_SMD:LED_0402_1005Metric, symbol Device:LED
- added IC3: LT8631IFE#PBF, SamacSys_Parts:SOP65P640X120-21N, symbol SamacSys_Parts:LT8631IFE#PBF
- added L1: 22uH Shld 20% 1.9A MSD1048-223MED, Inductor_SMD:L_Bourns_SRP1038C_10.0x10.0mm, symbol Device:L
- added R110, R111: 2.2k, Resistor_SMD:R_0805_2012Metric, symbol Device:R
- added R51: 75k, Resistor_SMD:R_0402_1005Metric, symbol Device:R
- added R52: 10k, Resistor_SMD:R_0402_1005Metric, symbol Device:R
- added R53: 8.66k, Resistor_SMD:R_0402_1005Metric, symbol Device:R
- added R56: 475k 1%, Resistor_SMD:R_0402_1005Metric, symbol Device:R
- added R57: 90.7k 1%, Resistor_SMD:R_0402_1005Metric, symbol Device:R
Connections:
- net 12V: now also C3.1, C64.1, IC3.1 (VIN), R110.1, R51.1
- net PwrGnd: now also C3.2, C64.2, C65.2, C66.2, C69.1, C70.2, IC3.13 (NC_3), IC3.15 (NC_4), IC3.21 (GND), IC3.6 (NC_1), IC3.7 (SYNC/MODE), IC3.9 (NC_2), R52.2, R53.2, R57.2
- new net: D5.1 (K), IC3.5 (PG)
- new net: D5.2 (A), R111.2
- new net: C67.1, IC3.20 (SW), L1.1
- new net: C67.2, IC3.18 (BST)
- new net: IC3.8 (RT), R53.1
- new net: C66.1, IC3.16 (INTVCC)
- new net: C65.1, IC3.10 (TR/SS)
- new net: C68.2, IC3.11 (FB), R56.2, R57.1
- new net: IC3.14 (IND), L1.2
- new net: R110.2, R111.1
- new net 5V: C68.1, C69.2, C70.1, IC3.12 (VOUT), R56.1
- new net EN: IC3.3 (EN/UV), R51.2, R52.1

Commit message: progress
Parts:
- C9: renamed from C3; footprint CAPAE1360X1450N -> SamacSys_Parts:CAPAE1360X1450N
- renumbered C64 to C10, C65 to C11, C66 to C12, C67 to C13, C68 to C14, C69 to C15, C70 to C16, IC3 to IC1, R110 to R41, R111 to R42, R51 to R43, R52 to R44, R53 to R45, R56 to R46, R57 to R47
Changed lines of the file:
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@@
 		(dnp no)
 		(fields_autoplaced yes)
-		(property "Reference" "C67"
+		(property "Reference" "C13"
 			(at 193.04 80.0099 0)
 			(show_name no)
@@
 			(project "kiln"
 				(path "/e9c1836b-d16f-494a-819b-41549a786e18/0dba9547-3e07-4b05-b251-0d0918aca780"
-					(reference "C67")
+					(reference "C13")
 					(unit 1)
 				)
@@
 		(dnp no)
 		(fields_autoplaced yes)
-		(property "Reference" "R53"
+		(property "Reference" "R45"
 			(at 124.46 109.2199 0)
 			(show_name no)
@@
 			(project "kiln"
 				(path "/e9c1836b-d16f-494a-819b-41549a786e18/0dba9547-3e07-4b05-b251-0d0918aca780"
-					(reference "R53")
+					(reference "R45")
 					(unit 1)
 				)
@@
 		(in_pos_files yes)
 		(dnp no)
-		(property "Reference" "C66"
+		(property "Reference" "C12"
 			(at 174.498 110.744 0)
 			(show_name no)
@@
 			(project "kiln"
 				(path "/e9c1836b-d16f-494a-819b-41549a786e18/0dba9547-3e07-4b05-b251-0d0918aca780"
-					(reference "C66")
+					(reference "C12")
 					(unit 1)
 				)
@@
 		(dnp no)
 		(fields_autoplaced yes)
-		(property "Reference" "C70"
+		(property "Reference" "C16"
 			(at 238.76 110.4899 0)
 			(show_name no)
@@
 			(project "kiln"
 				(path "/e9c1836b-d16f-494a-819b-41549a786e18/0dba9547-3e07-4b05-b251-0d0918aca780"
-					(reference "C70")
+					(reference "C16")
 					(unit 1)
 				)
@@
 		(dnp no)
 		(fields_autoplaced yes)
-		(property "Reference" "C65"
+		(property "Reference" "C11"
 			(at 135.89 114.2999 0)
 			(show_name no)
@@
 			(project "kiln"
 				(path "/e9c1836b-d16f-494a-819b-41549a786e18/0dba9547-3e07-4b05-b251-0d0918aca780"
-					(reference "C65")
+					(reference "C11")
 					(unit 1)
 				)
@@
 		(dnp no)
 		(fields_autoplaced yes)
-		(property "Reference" "R57"
+		(property "Reference" "R47"
 			(at 208.28 116.8399 0)
 			(show_name no)
@@
 			(project "kiln"
 				(path "/e9c1836b-d16f-494a-819b-41549a786e18/0dba9547-3e07-4b05-b251-0d0918aca780"
-					(reference "R57")
+					(reference "R47")
 					(unit 1)
 				)
@@
 		(dnp no)
 		(fields_autoplaced yes)
-		(property "Reference" "C68"
+		(property "Reference" "C14"
 			(at 196.85 105.4099 0)
 			(show_name no)
@@
 			(project "kiln"
 				(path "/e9c1836b-d16f-494a-819b-41549a786e18/0dba9547-3e07-4b05-b251-0d0918aca780"
-					(reference "C68")
+					(reference "C14")
 					(unit 1)
 				)
@@
 		(dnp yes)
 		(fields_autoplaced yes)
-		(property "Reference" "R52"
+		(property "Reference" "R44"
 			(at 121.92 80.0099 0)
 			(show_name no)
@@
 			(project "kiln"
 				(path "/e9c1836b-d16f-494a-819b-41549a786e18/0dba9547-3e07-4b05-b251-0d0918aca780"
-					(reference "R52")
+					(reference "R44")
 					(unit 1)
 				)
@@
 		(dnp no)
 		(fields_autoplaced yes)
-		(property "Reference" "R56"
+		(property "Reference" "R46"
 			(at 208.28 106.6799 0)
 			(show_name no)
@@
 			(project "kiln"
 				(path "/e9c1836b-d16f-494a-819b-41549a786e18/0dba9547-3e07-4b05-b251-0d0918aca780"
-					(reference "R56")
+					(reference "R46")
 					(unit 1)
 				)
@@
 		(dnp no)
 		(fields_autoplaced yes)
-		(property "Reference" "IC3"
+		(property "Reference" "IC1"
 			(at 156.21 73.66 0)
 			(show_name no)
@@
 			(project "kiln"
 				(path "/e9c1836b-d16f-494a-819b-41549a786e18/0dba9547-3e07-4b05-b251-0d0918aca780"
-					(reference "IC3")
+					(reference "IC1")
 					(unit 1)
 				)
@@
 		(dnp no)
 		(fields_autoplaced yes)
-		(property "Reference" "R51"
+		(property "Reference" "R43"
 			(at 121.92 69.8499 0)
 			(show_name no)
@@
 			(project "kiln"
 				(path "/e9c1836b-d16f-494a-819b-41549a786e18/0dba9547-3e07-4b05-b251-0d0918aca780"
-					(reference "R51")
+					(reference "R43")
 					(unit 1)
 				)
@@
 		(dnp no)
 		(fields_autoplaced yes)
-		(property "Reference" "R111"
+		(property "Reference" "R42"
 			(at 91.44 90.1699 0)
 			(show_name no)
@@
 			(project "kiln"
 				(path "/e9c1836b-d16f-494a-819b-41549a786e18/0dba9547-3e07-4b05-b251-0d0918aca780"
-					(reference "R111")
+					(reference "R42")
 					(unit 1)
 				)
@@
 		(in_pos_files yes)
 		(dnp no)
-		(property "Reference" "C69"
+		(property "Reference" "C15"
 			(at 218.694 112.268 90)
 			(show_name no)
@@
 			(project "kiln"
 				(path "/e9c1836b-d16f-494a-819b-41549a786e18/0dba9547-3e07-4b05-b251-0d0918aca780"
-					(reference "C69")
+					(reference "C15")
 					(unit 1)
 				)
@@
 		(in_pos_files yes)
 		(dnp no)
-		(property "Reference" "C3"
+		(property "Reference" "C9"
 			(at 97.79 71.1199 90)
 			(show_name no)
@@
 			)
 		)
-		(property "Footprint" "CAPAE1360X1450N"
+		(property "Footprint" "SamacSys_Parts:CAPAE1360X1450N"
 			(at 95.25 74.93 0)
 			(hide yes)
@@
 			(project "kiln"
 				(path "/e9c1836b-d16f-494a-819b-41549a786e18/0dba9547-3e07-4b05-b251-0d0918aca780"
-					(reference "C3")
+					(reference "C9")
 					(unit 1)
 				)
@@
 		(dnp no)
 		(fields_autoplaced yes)
-		(property "Reference" "R110"
+		(property "Reference" "R41"
 			(at 91.44 81.2799 0)
 			(show_name no)
@@
 			(project "kiln"
 				(path "/e9c1836b-d16f-494a-819b-41549a786e18/0dba9547-3e07-4b05-b251-0d0918aca780"
-					(reference "R110")
+					(reference "R41")
 					(unit 1)
 				)
@@
 		(dnp no)
 		(fields_autoplaced yes)
-		(property "Reference" "C64"
+		(property "Reference" "C10"
 			(at 111.76 69.8499 0)
 			(show_name no)
@@
 			(project "kiln"
 				(path "/e9c1836b-d16f-494a-819b-41549a786e18/0dba9547-3e07-4b05-b251-0d0918aca780"
-					(reference "C64")
+					(reference "C10")
 					(unit 1)
 				)

Commit message: add mouser sch tooling
Parts:
- C9: value 470uf 50v -> 470uf
- R47: value 90.7k 1% -> 90.9k 1%
Changed lines of the file:
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@@
 			)
 		)
-		(property "Value" "90.7k 1%"
+		(property "Value" "90.9k 1%"
 			(at 208.28 119.3799 0)
 			(show_name no)
@@
 			)
 		)
-		(property "Datasheet" "https://www.mouser.com/ProductDetail/Vishay/CRCW040247K5FKED?qs=sGAEpiMZZMtlubZbdhIBIPs%252BiE%2F4M15xDan5FFmucgw%3D"
+		(property "Datasheet" "https://www.mouser.com/en/ProductDetail/Vishay/CRCW040290K9FKED?qs=sGAEpiMZZMtlubZbdhIBIAbDPbIXdjYGA3h5w11HIuU%3D"
 			(at 205.74 118.11 0)
 			(hide yes)
@@
 			)
 		)
-		(property "Value" "470uf 50v"
+		(property "Value" "470uf"
 			(at 95.25 75.692 90)
 			(show_name no)

Commit message: more tooling and updateing of the sch
Parts:
- C15: Mouser https://www.mouser.com/ProductDetail/Murata-Electronics/GRM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 -> https://www.mouser.com/en/ProductDetail/Samsung-Electro-Mec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
Changed lines of the file:
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@@
 			)
 		)
-		(property "Datasheet" "https://www.mouser.com/datasheet/2/281/1/GRM32EC81C476KE15_01A-1988154.pdf"
+		(property "Datasheet" "https://www.mouser.com/en/ProductDetail/Samsung-Electro-Mechanics/CL32A476KOJNNNE?qs=d72FGnIDsgQXYP%252BbBe7Sww%3D%3D"
 			(at 222.25 110.49 0)
 			(hide yes)
@@
 			)
 		)
-		(property "Mouser" "https://www.mouser.com/ProductDetail/Murata-Electronics/GRM32EC81C476KE15L?qs=eeBpzGFlv%252B%2F0ttt4zOip7g%3D%3D"
+		(property "Mouser" "https://www.mouser.com/en/ProductDetail/Samsung-Electro-Mechanics/CL32A476KOJNNNE?qs=d72FGnIDsgQXYP%252BbBe7Sww%3D%3D"
 			(at 222.25 110.49 90)
 			(hide yes)

Commit message: start adding seprate Thermocouple Board, fix some errors
Parts:
- C10, C12: Mouser Part Number Alt (none) -> https://www.mouser.com/en/ProductDetail/Samsung-Electro-Mec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; Mouser Part Number Alt 2 (none) -> https://www.mouser.com/en/ProductDetail/Murata-Electronics/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; Mouser Part Number Alt 3 (none) -> https://www.mouser.com/en/ProductDetail/Murata-Electronics/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; Mouser Part Number Alt 4 (none) -> https://www.mouser.com/en/ProductDetail/KEMET/C1206C225K5RA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
Changed lines of the file:
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@@
+			)
+		)
+		(property "Mouser Part Number Alt 4" "https://www.mouser.com/en/ProductDetail/KEMET/C1206C225K5RACAUTO7210?qs=%252BfJPIY6s7PlNVZKyV3SAGA%3D%3D"
+			(at 179.07 113.03 0)
+			(hide yes)
+			(show_name no)
+			(do_not_autoplace no)
+			(effects
+				(font
+					(size 1.27 1.27)
+				)
+			)
+		)
+		(property "Mouser Part Number Alt 3" "https://www.mouser.com/en/ProductDetail/Murata-Electronics/GCM31CR71H225KA55L?qs=aEuGZpxfbxXH69FledLqTA%3D%3D"
+			(at 179.07 113.03 0)
+			(hide yes)
+			(show_name no)
+			(do_not_autoplace no)
+			(effects
+				(font
+					(size 1.27 1.27)
+				)
+			)
+		)
+		(property "Mouser Part Number Alt 2" "https://www.mouser.com/en/ProductDetail/Murata-Electronics/GRT31CR71H225KE13L?qs=qkDYIeTQ%252BEkhrDhfEIGgfg%3D%3D"
+			(at 179.07 113.03 0)
+			(hide yes)
+			(show_name no)
+			(do_not_autoplace no)
+			(effects
+				(font
+					(size 1.27 1.27)
+				)
+			)
+		)
+		(property "Mouser Part Number Alt" "https://www.mouser.com/en/ProductDetail/Samsung-Electro-Mechanics/CL31B225KBHNFNE?qs=%252B6g0mu59x7Ixea%2FwRKCoRw%3D%3D"
+			(at 179.07 113.03 0)
+			(hide yes)
+			(show_name no)
+			(do_not_autoplace no)
+			(effects
+				(font
+					(size 1.27 1.27)
+				)
 			)
 		)
@@
 			(at 107.95 71.12 0)
 			(hide yes)
+			(show_name no)
+			(do_not_autoplace no)
+			(effects
+				(font
+					(size 1.27 1.27)
+				)
+			)
+		)
+		(property "Mouser Part Number Alt 4" "https://www.mouser.com/en/ProductDetail/KEMET/C1206C225K5RACAUTO7210?qs=%252BfJPIY6s7PlNVZKyV3SAGA%3D%3D"
+			(at 107.95 71.12 0)
+			(hide yes)
+			(show_name no)
+			(do_not_autoplace no)
+			(effects
+				(font
+					(size 1.27 1.27)
+				)
+			)
+		)
+		(property "Mouser Part Number Alt 3" "https://www.mouser.com/en/ProductDetail/Murata-Electronics/GCM31CR71H225KA55L?qs=aEuGZpxfbxXH69FledLqTA%3D%3D"
+			(at 107.95 71.12 0)
+			(hide yes)
+			(show_name no)
+			(do_not_autoplace no)
+			(effects
+				(font
+					(size 1.27 1.27)
+				)
+			)
+		)
+		(property "Mouser Part Number Alt 2" "https://www.mouser.com/en/ProductDetail/Murata-Electronics/GRT31CR71H225KE13L?qs=qkDYIeTQ%252BEkhrDhfEIGgfg%3D%3D"
+			(at 107.95 71.12 0)
+			(hide yes)
+			(show_name no)
+			(do_not_autoplace no)
+			(effects
+				(font
+					(size 1.27 1.27)
+				)
+			)
+		)
+		(property "Mouser Part Number Alt" "https://www.mouser.com/en/ProductDetail/Samsung-Electro-Mechanics/CL31B225KBHNFNE?qs=%252B6g0mu59x7Ixea%2FwRKCoRw%3D%3D"
+			(at 107.95 71.12 0)
+			(hide yes)
