File: ThermocoupleBoard/ThermocoupleBoard.kicad_pcb (KiCad board)
At the start: 4 copper layers, 54 parts, among them J5 1935161, U6 MAX31856

Commit message: progress
Parts:
- added C1: 47uF 16V, Capacitor_SMD:C_1210_3225Metric, B.Cu at (77.7, 109.9)
- added C2: 0.01uf, Capacitor_SMD:C_0402_1005Metric, B.Cu at (81.9, 106.0)
- added C28: 47uF 16V, Capacitor_SMD:C_1210_3225Metric, F.Cu at (80.7, 109.9)
- added C3: 47uF 16V, Capacitor_SMD:C_1210_3225Metric, B.Cu at (84.5, 105.8)
- added J5: Conn_01x20_Pin, Connector_PinHeader_2.54mm:PinHeader_1x20_P2.54mm_Horizontal, F.Cu at (69.7, 96.9)
- added R1: 0, Resistor_SMD:R_0402_1005Metric, B.Cu at (81.9, 103.7)
- added R2: 0, Resistor_SMD:R_0402_1005Metric, B.Cu at (80.5, 103.1)
- added U1: LT1962-3.3, Package_SO:MSOP-8_3x3mm_P0.65mm, B.Cu at (77.7, 106.0)
- R10, R4, R7: renamed from R49; value 2k -> 2.2k
- R11, R5, R8: renamed from R50; value 2k -> 2.2k
- R3, R6, R9: renamed from R48; value 2k -> 2.2k
- moved C12 28.1 mm to (109.3, 126.7)
- moved C14 28.1 mm to (105.3, 126.7)
- moved C15 28.1 mm to (107.8, 125.7)
- moved C17 28.1 mm to (107.3, 123.2)
- moved C19 28.1 mm to (107.3, 122.2)
- moved FB5 28.1 mm to (108.8, 129.7)
- moved FB6 28.1 mm to (105.8, 129.7)
- moved R6 28.1 mm to (108.8, 128.2)
- moved R7 28.1 mm to (105.8, 128.2)
- moved R8 28.1 mm to (107.3, 127.7)
- moved U3 28.1 mm to (107.8, 121.2)
- moved D2 28.1 mm to (107.4, 131.7)
- moved FB7 28.1 mm to (108.8, 121.4)
- moved C16 28.1 mm to (111.3, 121.2)
- moved FB8 28.1 mm to (107.8, 120.5)
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- renumbered C73 to C10, C22 to C11, C17 to C12, C18 to C13, C19 to C14, C20 to C15, C69 to C16, C21 to C17, C73 to C18, C22 to C19, C17 to C20, C18 to C21, C19 to C22, C20 to C23, C69 to C24, C21 to C25, C73 to C26, C22 to C27, C17 to C4, C18 to C5, C19 to C6, C20 to C7, C69 to C8, C21 to C9, D28 to D1, D28 to D2, D28 to D3, FB2 to FB10, FB9 to FB11, FB13 to FB12, FB9 to FB3, FB13 to FB4, FB1 to FB5, FB2 to FB6, FB9 to FB7, FB13 to FB8, FB1 to FB9, J5 to J2, J5 to J3, J5 to J4, U6 to U2, U6 to U3, U6 to U4
Connections:
- net /SaftyProcessor/CLK renamed /CLK
- net /SaftyProcessor/MISO renamed /MISO
- net /SaftyProcessor/MOSI renamed /MOSI
- net GND_Safty renamed GND
- C10 pad 1: Net-(U6-DVDD) -> Net-(U2-DVDD)
- C11 pad 1: Net-(U6-DVDD) -> Net-(U2-DVDD)
- C12 pad 2: Net-(U6-T+) -> Net-(U3-T+)
- C13 pad 1: Net-(U6-T+) -> Net-(U3-T+)
- C13 pad 2: Net-(U6-T-) -> Net-(U3-T-)
- C14 pad 1: Net-(U6-T-) -> Net-(U3-T-)
- C15 pad 1: Net-(U6-BIAS) -> Net-(U3-BIAS)
- C16 pad 1: Net-(U6-AVDD) -> Net-(U3-AVDD)
- C17 pad 1: Net-(U6-AVDD) -> Net-(U3-AVDD)
- C18 pad 1: Net-(U6-DVDD) -> Net-(U3-DVDD)
- C19 pad 1: Net-(U6-DVDD) -> Net-(U3-DVDD)
- C20 pad 2: Net-(U6-T+) -> Net-(U4-T+)
- C21 pad 1: Net-(U6-T+) -> Net-(U4-T+)
- C21 pad 2: Net-(U6-T-) -> Net-(U4-T-)
- C22 pad 1: Net-(U6-T-) -> Net-(U4-T-)
- C23 pad 1: Net-(U6-BIAS) -> Net-(U4-BIAS)
- C24 pad 1: Net-(U6-AVDD) -> Net-(U4-AVDD)
- C25 pad 1: Net-(U6-AVDD) -> Net-(U4-AVDD)
- C26 pad 1: Net-(U6-DVDD) -> Net-(U4-DVDD)
- C27 pad 1: Net-(U6-DVDD) -> Net-(U4-DVDD)
- C4 pad 2: Net-(U6-T+) -> Net-(U2-T+)
- C5 pad 1: Net-(U6-T+) -> Net-(U2-T+)
- C5 pad 2: Net-(U6-T-) -> Net-(U2-T-)
- C6 pad 1: Net-(U6-T-) -> Net-(U2-T-)
- C7 pad 1: Net-(U6-BIAS) -> Net-(U2-BIAS)
- C8 pad 1: Net-(U6-AVDD) -> Net-(U2-AVDD)
- C9 pad 1: Net-(U6-AVDD) -> Net-(U2-AVDD)
- D1 pad 1: Net-(D28-K-Pad1) -> Net-(D1-K-Pad1)
- D1 pad 2: Net-(D28-K-Pad2) -> Net-(D1-K-Pad2)
- D2 pad 1: Net-(D28-K-Pad1) -> Net-(D2-K-Pad1)
- D2 pad 2: Net-(D28-K-Pad2) -> Net-(D2-K-Pad2)
- D3 pad 1: Net-(D28-K-Pad1) -> Net-(D3-K-Pad1)
- D3 pad 2: Net-(D28-K-Pad2) -> Net-(D3-K-Pad2)
- FB1 pad 2: Net-(D28-K-Pad1) -> Net-(D1-K-Pad1)
- FB10 pad 1: Net-(FB2-Pad1) -> Net-(FB10-Pad1)
- FB10 pad 2: Net-(D28-K-Pad2) -> Net-(D3-K-Pad2)
- FB11 pad 1: Net-(U6-AVDD) -> Net-(U4-AVDD)
- FB11 pad 2: 3.3v_Safty -> 3.3V_A
- FB12 pad 1: Net-(U6-DVDD) -> Net-(U4-DVDD)
- FB12 pad 2: 3.3v_Safty -> 3.3_D
- FB2 pad 2: Net-(D28-K-Pad2) -> Net-(D1-K-Pad2)
- FB3 pad 1: Net-(U6-AVDD) -> Net-(U2-AVDD)
- FB3 pad 2: 3.3v_Safty -> 3.3V_A
- FB4 pad 1: Net-(U6-DVDD) -> Net-(U2-DVDD)
- FB4 pad 2: 3.3v_Safty -> 3.3_D
- FB5 pad 1: Net-(FB1-Pad1) -> Net-(FB5-Pad1)
- FB5 pad 2: Net-(D28-K-Pad1) -> Net-(D2-K-Pad1)
- FB6 pad 1: Net-(FB2-Pad1) -> Net-(FB6-Pad1)
- FB6 pad 2: Net-(D28-K-Pad2) -> Net-(D2-K-Pad2)
- FB7 pad 1: Net-(U6-AVDD) -> Net-(U3-AVDD)
- FB7 pad 2: 3.3v_Safty -> 3.3V_A
- FB8 pad 1: Net-(U6-DVDD) -> Net-(U3-DVDD)
- FB8 pad 2: 3.3v_Safty -> 3.3_D
- FB9 pad 1: Net-(FB1-Pad1) -> Net-(FB9-Pad1)
- FB9 pad 2: Net-(D28-K-Pad1) -> Net-(D3-K-Pad1)
- J3 pad 1: Net-(FB2-Pad1) -> Net-(FB6-Pad1)
- J3 pad 2: Net-(FB1-Pad1) -> Net-(FB5-Pad1)
- J4 pad 1: Net-(FB2-Pad1) -> Net-(FB10-Pad1)
- J4 pad 2: Net-(FB1-Pad1) -> Net-(FB9-Pad1)
- R10 pad 1: Net-(U6-T-) -> Net-(U4-T-)
- R10 pad 2: Net-(D28-K-Pad2) -> Net-(D3-K-Pad2)
- R11 pad 1: Net-(U6-BIAS) -> Net-(U4-BIAS)
- R11 pad 2: Net-(D28-K-Pad2) -> Net-(D3-K-Pad2)
- R3 pad 1: Net-(U6-T+) -> Net-(U2-T+)
- R3 pad 2: Net-(D28-K-Pad1) -> Net-(D1-K-Pad1)
- R4 pad 1: Net-(U6-T-) -> Net-(U2-T-)
- R4 pad 2: Net-(D28-K-Pad2) -> Net-(D1-K-Pad2)
- R5 pad 1: Net-(U6-BIAS) -> Net-(U2-BIAS)
- R5 pad 2: Net-(D28-K-Pad2) -> Net-(D1-K-Pad2)
- R6 pad 1: Net-(U6-T+) -> Net-(U3-T+)
- R6 pad 2: Net-(D28-K-Pad1) -> Net-(D2-K-Pad1)
- R7 pad 1: Net-(U6-T-) -> Net-(U3-T-)
- R7 pad 2: Net-(D28-K-Pad2) -> Net-(D2-K-Pad2)
- R8 pad 1: Net-(U6-BIAS) -> Net-(U3-BIAS)
- R8 pad 2: Net-(D28-K-Pad2) -> Net-(D2-K-Pad2)
- R9 pad 1: Net-(U6-T+) -> Net-(U4-T+)
- R9 pad 2: Net-(D28-K-Pad1) -> Net-(D3-K-Pad1)
- U2 pad 13: /SaftyProcessor/thermoFault -> /thermoFault_0
- U2 pad 2: Net-(U6-BIAS) -> Net-(U2-BIAS)
- U2 pad 3: Net-(U6-T-) -> Net-(U2-T-)
- U2 pad 4: Net-(U6-T+) -> Net-(U2-T+)
- U2 pad 5: Net-(U6-AVDD) -> Net-(U2-AVDD)
- U2 pad 6: unconnected-(U6-DNC-Pad6) -> unconnected-(U2-DNC-Pad6)
- U2 pad 7: /SaftyProcessor/thermoDrdy -> /thermoDrdy_0
- U2 pad 8: Net-(U6-DVDD) -> Net-(U2-DVDD)
- U2 pad 9: /SaftyProcessor/CS0 -> /CS0
- U3 pad 13: /SaftyProcessor/thermoFault -> /thermoFault_1
- U3 pad 2: Net-(U6-BIAS) -> Net-(U3-BIAS)
- U3 pad 3: Net-(U6-T-) -> Net-(U3-T-)
- U3 pad 4: Net-(U6-T+) -> Net-(U3-T+)
- U3 pad 5: Net-(U6-AVDD) -> Net-(U3-AVDD)
- U3 pad 6: unconnected-(U6-DNC-Pad6) -> unconnected-(U3-DNC-Pad6)
- U3 pad 7: /SaftyProcessor/thermoDrdy -> /thermoDrdy_1
- U3 pad 8: Net-(U6-DVDD) -> Net-(U3-DVDD)
- U3 pad 9: /SaftyProcessor/CS0 -> /CS1
- U4 pad 13: /SaftyProcessor/thermoFault -> /thermoFault_2
- U4 pad 2: Net-(U6-BIAS) -> Net-(U4-BIAS)
- U4 pad 3: Net-(U6-T-) -> Net-(U4-T-)
- U4 pad 4: Net-(U6-T+) -> Net-(U4-T+)
- U4 pad 5: Net-(U6-AVDD) -> Net-(U4-AVDD)
- U4 pad 6: unconnected-(U6-DNC-Pad6) -> unconnected-(U4-DNC-Pad6)
- U4 pad 7: /SaftyProcessor/thermoDrdy -> /thermoDrdy_2
- U4 pad 8: Net-(U6-DVDD) -> Net-(U4-DVDD)
- U4 pad 9: /SaftyProcessor/CS0 -> /CS2
Routing:
- net 3.3V_A: track 0.00 -> 59.4 mm, vias 0 -> 5
- net 3.3_D: track 0.00 -> 57.5 mm, vias 0 -> 6
- net /MISO: track 8.94 -> 58.5 mm, vias 0 -> 4
- net /MOSI: track 11.5 -> 59.4 mm, vias 0 -> 2
- net /CLK: track 12.2 -> 59.8 mm, vias 0 -> 2
- net /thermoDrdy_1: track 0.00 -> 47.5 mm, vias 0 -> 1
- net /thermoFault_0: track 0.00 -> 44.0 mm, vias 0 -> 2
- net /thermoDrdy_0: track 0.00 -> 43.2 mm, vias 0 -> 1
- net /CS2: track 0.00 -> 39.6 mm, vias 0 -> 2
- net /thermoFault_1: track 0.00 -> 37.7 mm, vias 0 -> 1
- net /SaftyProcessor/thermoDrdy: track 30.9 -> 0.00 mm
- net Net-(U6-DVDD): track 30.5 -> 0.00 mm, vias 3 -> 0
- net /thermoDrdy_2: track 0.00 -> 29.0 mm, vias 0 -> 2
- net /thermoFault_2: track 0.00 -> 25.2 mm
- net /CS1: track 0.00 -> 24.3 mm, vias 0 -> 2
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- added copper zone on B.Cu, net GND
- added copper zone on F.Cu, net GND
- added copper zone on In1.Cu, net GND
Other:
- board outline added: 51.2 x 49.9 mm
