File: ThermocoupleBoard/ThermocoupleBoard.kicad_sch (KiCad schematic)
At the start: 7 parts, among them J1 Conn_01x16_Pin, U1 LT1962-3.3

Commit message: sch update
Connections:
- net GND: no longer J1.14 (Pin_14)
- net SCL: now reaches J1.15 (Pin_15)
- new net SDA: J1.14 (Pin_14)
Changed lines of the file:
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@@
 	(paper "A4")
-	(junction
-		(at 222.25 88.9)
-		(diameter 0)
-		(color 0 0 0 0)
-	)
 	(junction
 		(at 222.25 93.98)
@@
 	(wire
 		(pts
+			(xy 200.66 88.9) (xy 224.79 88.9)
+		)
+		(stroke
+			(width 0)
+			(type default)
+		)
+	)
+	(wire
+		(pts
 			(xy 200.66 83.82) (xy 224.79 83.82)
 		)
@@
 	(wire
 		(pts
-			(xy 222.25 76.2) (xy 222.25 88.9)
-		)
-		(stroke
-			(width 0)
-			(type default)
-		)
-	)
-	(wire
-		(pts
 			(xy 41.91 100.33) (xy 41.91 99.06)
 		)
@@
 	(wire
 		(pts
-			(xy 222.25 88.9) (xy 224.79 88.9)
-		)
-		(stroke
-			(width 0)
-			(type default)
-		)
-	)
-	(wire
-		(pts
 			(xy 83.82 116.84) (xy 85.09 116.84)
 		)
@@
 	(wire
 		(pts
+			(xy 200.66 91.44) (xy 224.79 91.44)
+		)
+		(stroke
+			(width 0)
+			(type default)
+		)
+	)
+	(wire
+		(pts
 			(xy 41.91 99.06) (xy 46.99 99.06)
 		)
@@
 	(wire
 		(pts
-			(xy 222.25 88.9) (xy 222.25 93.98)
+			(xy 222.25 76.2) (xy 222.25 93.98)
 		)
 		(stroke
@@
 		)
 	)
+	(label "SDA"
+		(at 200.66 88.9 0)
+		(effects
+			(font
+				(size 1.27 1.27)
+			)
+			(justify left bottom)
+		)
+	)
 	(label "CS0"
 		(at 87.63 63.5 0)
@@
 	(label "CS2"
 		(at 200.66 86.36 0)
+		(effects
+			(font
+				(size 1.27 1.27)
+			)
+			(justify left bottom)
+		)
+	)
+	(label "SCL"
+		(at 200.66 91.44 0)
 		(effects
 			(font
@@
 			)
 		)
+		(property "Description" "Generic connector, single row, 01x16, script generated"
+			(at 229.87 73.66 0)
+			(hide yes)
+			(show_name no)
+			(do_not_autoplace no)
+			(effects
+				(font
+					(size 1.27 1.27)
+				)
+			)
+		)
 		(property "Mouser Part Number Alt 2" "https://www.mouser.com/en/ProductDetail/Amphenol-FCI/68016-116HLF?qs=QKvFUfBIyQJGaW1tNFNciA%3D%3D"
 			(at 229.87 73.66 0)
@@
 			(at 229.87 73.66 0)
 			(hide yes)
-			(show_name no)
-			(do_not_autoplace no)
-			(effects
-				(font
-					(size 1.27 1.27)
-				)
-			)
-		)
-		(property "Description" "Generic connector, single row, 01x16, script generated"
-			(at 229.87 73.66 0)
-			(hide yes)

Commit message: progress
Parts:
- removed J1: Conn_01x16_Pin, Connector_PinHeader_2.54mm:PinHeader_1x16_P2.54mm_Horizontal, symbol Connector:Conn_01x16_Pin
- added C28: 47uF 16V, Capacitor_SMD:C_1210_3225Metric, symbol Device:C
- added J5: Conn_01x20_Pin, Connector_PinHeader_2.54mm:PinHeader_1x20_P2.54mm_Horizontal, symbol Connector:Conn_01x20_Pin
Connections:
- net 3.3_D: now also C28.2
- net 5V: now also J5.1 (Pin_1)
- net CLK: now also J5.12 (Pin_12)
- net CS0: now also J5.13 (Pin_13)
- net CS1: now also J5.14 (Pin_14)
- net CS2: now also J5.15 (Pin_15)
- net GND: now also C28.1, J5.18 (Pin_18), J5.19 (Pin_19), J5.20 (Pin_20), J5.9 (Pin_9)
- net MISO: now also J5.11 (Pin_11)
- net MOSI: now also J5.10 (Pin_10)
- net SCL: now also J5.17 (Pin_17)
- net SDA: now also J5.16 (Pin_16)
- net thermoDrdy_0: now also J5.4 (Pin_4)
- net thermoDrdy_1: now also J5.6 (Pin_6)
- net thermoDrdy_2: now also J5.8 (Pin_8)
- net thermoFault_0: now also J5.3 (Pin_3)
- net thermoFault_1: now also J5.5 (Pin_5)
- net thermoFault_2: now also J5.7 (Pin_7)
- net at R2.2: now also J5.2 (Pin_2)
