File: mainBoard/kiln.kicad_pcb (KiCad board)
At the start: 4 copper layers, 203.1 x 114.5 mm, 217 parts, among them IC4 MAXM17572AMC+T, IC5 MAXM17572AMC+T, IC6 MAXM17572AMC+T, IC7 MAXM17572AMC+T, J1 1935161, J10 1935174, J11 1935174, J12 1935161, J13 SJ2-35813B-SMT-TR, J14 1935161, J15 SJ2-35813B-SMT-TR, J16 1935161, J17 SJ2-35813B-SMT-TR, J18 1935161, J19 1935161, J2 Conn_01x10_Pin, J20 1935161, J21 1935161, J23 1935161, J24 1935161, J25 1935161, J3 1935174, J4 1935174, J6 Conn_01x20_Socket, J7 Conn_02x06_Odd_Even, J8 1935174, K1 EE2-12NUH, K2 EE2-12NUH, K3 EE2-12NUH, K4 EE2-12NUH, K5 EE2-12NUH, Q1 BSS138P,215, Q2 BSS138P,215, Q3 BSS138P,215, Q4 BSS138P,215, Q5 BSS138P,215, U1 TCMT1109, U10 LMV321, U11 LMV321, U12 LMV321, U13 TCMT1109, U14 TCMT1109, U2 TCMT1109, U3 TCMT1109, U4 ESP32-S3-DevKitC, U5 SX1509

Commit message: i think the pcbs and sch are good
Parts:
- C69, C70: value 6500p -> 6800p
- R35, R36, R39, R40, R59, R60, R66, R67, R70, R71: footprint Resistor_SMD:R_1206_3216Metric -> Resistor_SMD:R_2010_5025Metric
- moved R60 1.23 mm to (228.8, 58.3)
- moved R67 1.20 mm to (75.5, 83.9)
- moved R70 1.15 mm to (216.7, 58.2)
- moved R71 1.15 mm to (210.2, 58.2)
- moved R66 1.14 mm to (75.4, 77.6)
- moved R59 1.14 mm to (235.1, 58.2)
- moved R36 1.13 mm to (173.7, 58.2)
- moved R35 1.05 mm to (179.9, 58.1)
- moved R40 1.03 mm to (192.1, 58.1)
- moved R39 0.95 mm to (198.4, 58.0)
Routing:
- net 12V_Main: track 230.5 -> 168.8 mm, vias 28 -> 21
- net GND_Main: track 173.5 -> 137.6 mm, vias 250 -> 244
- net 3.3v_Safty: track 68.3 -> 76.9 mm, vias 32 -> 33
- net 12v_Safty: track 115.8 -> 108.3 mm, vias 18 -> 19
- net 3.3V_Main: track 137.9 -> 142.4 mm
- net Net-(J10-Pad1): track 34.4 -> 32.6 mm
- net /SaftyProcessor/estop: track 74.7 -> 76.4 mm
- net Net-(D9-A2): track 25.5 -> 24.4 mm
Other:
- outline, holes or cut-outs redrawn
