File: mainBoard/SSD.kicad_sch (KiCad schematic)
At the start: 10 parts, among them J3 1935174, K1 EE2-12NUH, Q1 BSS138P,215

Commit message: i think the pcbs and sch are good
Parts:
- R35, R36: footprint Resistor_SMD:R_1206_3216Metric -> Resistor_SMD:R_2010_5025Metric; Manufacturer_Name (none) -> Bourns; Manufacturer_Part_Number (none) -> CR2010-J/-000ELF; Mouser Part Number (none) -> https://www.mouser.com/en/ProductDetail/Bourns/CR2010-J-000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; Mouser Part Number Alt (none) -> https://www.mouser.com/en/ProductDetail/Vishay/CRCW20100000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; Mouser Part Number Alt 2 (none) -> https://www.mouser.com/en/ProductDetail/KOA-Speer/RK73Z2HTT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; Mouser Part Number Alt 3 (none) -> https://www.mouser.com/en/ProductDetail/Vishay/CRCW20100000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
Changed lines of the file:
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@@
 			)
 		)
-		(property "Footprint" "Resistor_SMD:R_1206_3216Metric"
+		(property "Footprint" "Resistor_SMD:R_2010_5025Metric"
 			(at 154.94 94.488 90)
 			(hide yes)
@@
 			)
 		)
-		(property "Datasheet" "https://www.mouser.com/ProductDetail/Royalohm/1206S4J0000TDE?qs=jcD%2FCkGBYePiYOBtSMuX2g%3D%3D"
+		(property "Datasheet" "https://www.mouser.com/en/ProductDetail/Bourns/CR2010-J-000ELF?qs=iQmVXIlZDPkUtxAs54Hu3Q%3D%3D"
 			(at 154.94 92.71 0)
 			(hide yes)
@@
 		)
 		(property "Description" "Resistor"
+			(at 154.94 92.71 0)
+			(hide yes)
+			(show_name no)
+			(do_not_autoplace no)
+			(effects
+				(font
+					(size 1.27 1.27)
+				)
+			)
+		)
+		(property "Mouser Part Number Alt 3" "https://www.mouser.com/en/ProductDetail/Vishay/CRCW20100000ZSTF?qs=LuV47j0yrcCuX3titWMqhw%3D%3D"
+			(at 154.94 92.71 0)
+			(hide yes)
+			(show_name no)
+			(do_not_autoplace no)
+			(effects
+				(font
+					(size 1.27 1.27)
+				)
+			)
+		)
+		(property "Mouser Part Number Alt 2" "https://www.mouser.com/en/ProductDetail/KOA-Speer/RK73Z2HTTE?qs=yjBPpuQqhAOWWHTNoHnqSQ%3D%3D"
+			(at 154.94 92.71 0)
+			(hide yes)
+			(show_name no)
+			(do_not_autoplace no)
+			(effects
+				(font
+					(size 1.27 1.27)
+				)
+			)
+		)
+		(property "Mouser Part Number Alt" "https://www.mouser.com/en/ProductDetail/Vishay/CRCW20100000Z0EF?qs=uSoEc56oFvrUbxXi0J%2Fe1w%3D%3D"
+			(at 154.94 92.71 0)
+			(hide yes)
+			(show_name no)
+			(do_not_autoplace no)
+			(effects
+				(font
+					(size 1.27 1.27)
+				)
+			)
+		)
+		(property "Mouser Part Number" "https://www.mouser.com/en/ProductDetail/Bourns/CR2010-J-000ELF?qs=iQmVXIlZDPkUtxAs54Hu3Q%3D%3D"
+			(at 154.94 92.71 0)
+			(hide yes)
+			(show_name no)
+			(do_not_autoplace no)
+			(effects
+				(font
+					(size 1.27 1.27)
+				)
+			)
+		)
+		(property "Manufacturer_Part_Number" "CR2010-J/-000ELF"
+			(at 154.94 92.71 0)
+			(hide yes)
+			(show_name no)
+			(do_not_autoplace no)
+			(effects
+				(font
+					(size 1.27 1.27)
+				)
+			)
+		)
+		(property "Manufacturer_Name" "Bourns"
 			(at 154.94 92.71 0)
 			(hide yes)
@@
 			)
 		)
-		(property "Footprint" "Resistor_SMD:R_1206_3216Metric"
+		(property "Footprint" "Resistor_SMD:R_2010_5025Metric"
 			(at 154.94 64.008 90)
 			(hide yes)
@@
 			)
 		)
-		(property "Datasheet" "https://www.mouser.com/ProductDetail/Royalohm/1206S4J0000TDE?qs=jcD%2FCkGBYePiYOBtSMuX2g%3D%3D"
+		(property "Datasheet" "https://www.mouser.com/en/ProductDetail/Bourns/CR2010-J-000ELF?qs=iQmVXIlZDPkUtxAs54Hu3Q%3D%3D"
 			(at 154.94 62.23 0)
 			(hide yes)
@@
 			(at 154.94 62.23 0)
 			(hide yes)
+			(show_name no)
+			(do_not_autoplace no)
+			(effects
+				(font
+					(size 1.27 1.27)
+				)
+			)
+		)
+		(property "Mouser Part Number Alt 3" "https://www.mouser.com/en/ProductDetail/Vishay/CRCW20100000ZSTF?qs=LuV47j0yrcCuX3titWMqhw%3D%3D"
+			(at 154.94 62.23 0)
+			(hide yes)
+			(show_name no)
+			(do_not_autoplace no)
+			(effects
+				(font
+					(size 1.27 1.27)
+				)
+			)
+		)
+		(property "Mouser Part Number Alt 2" "https://www.mouser.com/en/ProductDetail/KOA-Speer/RK73Z2HTTE?qs=yjBPpuQqhAOWWHTNoHnqSQ%3D%3D"
+			(at 154.94 62.23 0)
+			(hide yes)
+			(show_name no)
+			(do_not_autoplace no)
+			(effects
+				(font
+					(size 1.27 1.27)
+				)
+			)
+		)
+		(property "Mouser Part Number Alt" "https://www.mouser.com/en/ProductDetail/Vishay/CRCW20100000Z0EF?qs=uSoEc56oFvrUbxXi0J%2Fe1w%3D%3D"
+			(at 154.94 62.23 0)
+			(hide yes)
+			(show_name no)
+			(do_not_autoplace no)
+			(effects
+				(font
+					(size 1.27 1.27)
+				)
+			)
+		)
+		(property "Mouser Part Number" "https://www.mouser.com/en/ProductDetail/Bourns/CR2010-J-000ELF?qs=iQmVXIlZDPkUtxAs54Hu3Q%3D%3D"
+			(at 154.94 62.23 0)
+			(hide yes)
+			(show_name no)
+			(do_not_autoplace no)
+			(effects
+				(font
+					(size 1.27 1.27)
+				)
+			)
+		)
+		(property "Manufacturer_Part_Number" "CR2010-J/-000ELF"
+			(at 154.94 62.23 0)
+			(hide yes)
+			(show_name no)
+			(do_not_autoplace no)
+			(effects
+				(font
+					(size 1.27 1.27)
+				)
+			)
+		)
+		(property "Manufacturer_Name" "Bourns"
+			(at 154.94 62.23 0)
+			(hide yes)

Commit message: add a unit test fixture, and start changing the current measurement circuit
Connections:
- no-connect marks 0 -> 3
Changed lines of the file:
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@@
 		(color 0 0 0 0)
+	)
+	(no_connect
+		(at 151.13 73.66)
+	)
+	(no_connect
+		(at 153.67 88.9)
+	)
+	(no_connect
+		(at 156.21 73.66)
 	)
 	(wire
