File: mainBoard/SaftyProcessor.kicad_sch (KiCad schematic)
At the start: 20 parts, among them J1 1935161, U1 TCMT1109, U2 TCMT1109, U3 TCMT1109

Commit message: need to finish new regulators and run parts check on sch
Parts:
- added J7: Conn_02x06_Odd_Even, Connector_PinSocket_1.27mm:PinSocket_2x06_P1.27mm_Horizontal, symbol Connector_Generic:Conn_02x06_Odd_Even
- added R48, R49: 2.2k, Resistor_SMD:R_0402_1005Metric, symbol Device:R
- added R51: 0, Resistor_SMD:R_0402_1005Metric, symbol PCM_SparkFun-Resistor:R
Connections:
- net 3.3v_Safty: now also R48.2, R49.2, R51.1
- net CLK: now also J7.9 (Pin_9)
- net CS0: now also J7.11 (Pin_11)
- net GND_Safty: now also J7.10 (Pin_10), J7.12 (Pin_12)
- net MISO: now also J7.7 (Pin_7)
- net MOSI: now also J7.5 (Pin_5)
- net thermoDrdy: now also A1.16 (GPIO12), J7.4 (Pin_4); no longer A1.11 (GPIO8)
- net thermoFault: now also A1.15 (GPIO11), J7.3 (Pin_3); no longer A1.10 (GPIO7)
- new net: J7.1 (Pin_1), R51.2
- new net 5V: J7.2 (Pin_2)
- new net SCL: A1.11 (GPIO8), J7.8 (Pin_8), R49.1
- new net SDA: A1.10 (GPIO7), J7.6 (Pin_6), R48.1
Other:
- removed sheet SaftyThermocouple

Commit message: almost done
Connections:
- net 5V renamed 5v_Safty
Changed lines of the file:
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@@
 	(wire
 		(pts
+			(xy 127 166.37) (xy 127 163.83)
+		)
+		(stroke
+			(width 0)
+			(type default)
+		)
+	)
+	(wire
+		(pts
 			(xy 104.14 33.02) (xy 109.22 33.02)
 		)
@@
 	(wire
 		(pts
+			(xy 128.27 166.37) (xy 127 166.37)
+		)
+		(stroke
+			(width 0)
+			(type default)
+		)
+	)
+	(wire
+		(pts
 			(xy 43.18 120.65) (xy 43.18 123.19)
 		)
@@
 		)
 	)
+	(hierarchical_label "5V"
+		(shape input)
+		(at 128.27 166.37 0)
+		(effects
+			(font
+				(size 1.27 1.27)
+			)
+			(justify left)
+		)
+	)
 	(hierarchical_label "Gnd"
 		(shape passive)
@@
 	(symbol
 		(lib_id "power:VPP")
-		(at 58.42 127 0)
-		(unit 1)
-		(body_style 1)
-		(exclude_from_sim no)
-		(in_bom yes)
-		(on_board yes)
-		(in_pos_files yes)
-		(dnp no)
-		(fields_autoplaced yes)
-		(property "Reference" "#PWR031"
-			(at 58.42 130.81 0)
-			(hide yes)
-			(show_name no)
-			(do_not_autoplace no)
-			(effects
-				(font
-					(size 1.27 1.27)
-				)
-			)
-		)
-		(property "Value" "5V"
-			(at 58.42 121.92 0)
-			(show_name no)
-			(do_not_autoplace no)
-			(effects
-				(font
-					(size 1.27 1.27)
-				)
-			)
-		)
-		(property "Footprint" ""
-			(at 58.42 127 0)
-			(hide yes)
-			(show_name no)
-			(do_not_autoplace no)
-			(effects
-				(font
-					(size 1.27 1.27)
-				)
-			)
-		)
-		(property "Datasheet" ""
-			(at 58.42 127 0)
-			(hide yes)
-			(show_name no)
-			(do_not_autoplace no)
-			(effects
-				(font
-					(size 1.27 1.27)
-				)
-			)
-		)
-		(property "Description" "Power symbol creates a global label with name \"VPP\""
-			(at 58.42 127 0)
-			(hide yes)
-			(show_name no)
-			(do_not_autoplace no)
-			(effects
-				(font
-					(size 1.27 1.27)
-				)
-			)
-		)
-		(pin "1"
-		)
-		(instances
-			(project "kiln"
-				(path "/e9c1836b-d16f-494a-819b-41549a786e18/9d216770-eb40-4527-939f-01f0f376c505"
-					(reference "#PWR031")
-					(unit 1)
-				)
-			)
-		)
-	)
-	(symbol
-		(lib_id "power:VPP")
 		(at 233.68 27.94 0)
 		(unit 1)
@@
 					(unit 1)
 				)
+			)
+		)
+	)
+	(symbol
+		(lib_id "power:VPP")
+		(at 127 163.83 0)
+		(unit 1)
+		(body_style 1)
+		(exclude_from_sim no)
+		(in_bom yes)
+		(on_board yes)
+		(in_pos_files yes)
+		(dnp no)
+		(fields_autoplaced yes)
+		(property "Reference" "#PWR032"
+			(at 127 167.64 0)
+			(hide yes)
+			(show_name no)
+			(do_not_autoplace no)
+			(effects
+				(font
+					(size 1.27 1.27)
+				)
+			)
+		)
+		(property "Value" "5v_Safty"
+			(at 127 158.75 0)
+			(show_name no)
+			(do_not_autoplace no)
+			(effects
+				(font
+					(size 1.27 1.27)
+				)
+			)
+		)
+		(property "Footprint" ""
+			(at 127 163.83 0)
+			(hide yes)
+			(show_name no)
+			(do_not_autoplace no)
+			(effects
+				(font
+					(size 1.27 1.27)
+				)
+			)
+		)
+		(property "Datasheet" ""
+			(at 127 163.83 0)
+			(hide yes)
+			(show_name no)
+			(do_not_autoplace no)
+			(effects
+				(font
+					(size 1.27 1.27)
+				)
+			)
+		)
+		(property "Description" "Power symbol creates a global label with name \"VPP\""
+			(at 127 163.83 0)
+			(hide yes)
+			(show_name no)
+			(do_not_autoplace no)
+			(effects
+				(font
+					(size 1.27 1.27)
+				)
+			)
+		)
+		(pin "1"
+		)
+		(instances
+			(project "kiln"
+				(path "/e9c1836b-d16f-494a-819b-41549a786e18/9d216770-eb40-4527-939f-01f0f376c505"
+					(reference "#PWR032")
+					(unit 1)
+				)
+			)
+		)
+	)
+	(symbol
+		(lib_id "power:VPP")
+		(at 58.42 127 0)
+		(unit 1)
+		(body_style 1)
+		(exclude_from_sim no)
+		(in_bom yes)
+		(on_board yes)
+		(in_pos_files yes)
+		(dnp no)
+		(fields_autoplaced yes)
+		(property "Reference" "#PWR033"
+			(at 58.42 130.81 0)
+			(hide yes)
+			(show_name no)
+			(do_not_autoplace no)
+			(effects
+				(font
+					(size 1.27 1.27)
+				)
+			)
+		)
+		(property "Value" "5v_Safty"
+			(at 58.42 121.92 0)
+			(show_name no)
+			(do_not_autoplace no)
+			(effects
+				(font
+					(size 1.27 1.27)
+				)
+			)
+		)
+		(property "Footprint" ""
+			(at 58.42 127 0)
+			(hide yes)
+			(show_name no)
+			(do_not_autoplace no)
+			(effects
+				(font
+					(size 1.27 1.27)
+				)
+			)
+		)
+		(property "Datasheet" ""
+			(at 58.42 127 0)
+			(hide yes)
+			(show_name no)
+			(do_not_autoplace no)
+			(effects
+				(font
+					(size 1.27 1.27)
+				)
+			)
+		)
+		(property "Description" "Power symbol creates a global label with name \"VPP\""
+			(at 58.42 127 0)
+			(hide yes)
+			(show_name no)
+			(do_not_autoplace no)
+			(effects
+				(font
+					(size 1.27 1.27)
+				)
+			)
+		)
+		(pin "1"
+		)
+		(instances
+			(project "kiln"
+				(path "/e9c1836b-d16f-494a-819b-41549a786e18/9d216770-eb40-4527-939f-01f0f376c505"
+					(reference "#PWR033")
+					(unit 1)
+				)

Commit message: i think the pcbs and sch are good
Parts:
- R10, R8, R9: Manufacturer_Name (none) -> Vishay / Draloric; Manufacturer_Part_Number (none) -> RCS04021K00FKED; Mouser Part Number (none) -> https://www.mouser.com/en/ProductDetail/Vishay-Draloric/RCS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
Changed lines of the file:
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@@
 			)
 		)
-		(property "Datasheet" "https://www.mouser.com/ProductDetail/Vishay-Beyschlag/MCS04020C1001FE000?qs=sGAEpiMZZMtlubZbdhIBIMFZrYW9%252Bak7nVRDfe1Ameo%3D"
+		(property "Datasheet" "https://www.mouser.com/en/ProductDetail/Vishay-Draloric/RCS04021K00FKED?qs=NKmfXavxMazECCYilLNNOw%3D%3D"
+			(at 218.44 72.39 0)
+			(hide yes)
+			(show_name no)
+			(do_not_autoplace no)
+			(effects
+				(font
+					(size 1.27 1.27)
+				)
+			)
+		)
+		(property "Mouser Part Number" "https://www.mouser.com/en/ProductDetail/Vishay-Draloric/RCS04021K00FKED?qs=NKmfXavxMazECCYilLNNOw%3D%3D"
+			(at 218.44 72.39 0)
+			(hide yes)
+			(show_name no)
+			(do_not_autoplace no)
+			(effects
+				(font
+					(size 1.27 1.27)
+				)
+			)
+		)
+		(property "Manufacturer_Part_Number" "RCS04021K00FKED"
+			(at 218.44 72.39 0)
+			(hide yes)
+			(show_name no)
+			(do_not_autoplace no)
+			(effects
+				(font
+					(size 1.27 1.27)
+				)
+			)
+		)
+		(property "Manufacturer_Name" "Vishay / Draloric"
 			(at 218.44 72.39 0)
 			(hide yes)
@@
 			)
 		)
-		(property "Datasheet" "https://www.mouser.com/ProductDetail/Vishay-Beyschlag/MCS04020C1001FE000?qs=sGAEpiMZZMtlubZbdhIBIMFZrYW9%252Bak7nVRDfe1Ameo%3D"
+		(property "Datasheet" "https://www.mouser.com/en/ProductDetail/Vishay-Draloric/RCS04021K00FKED?qs=NKmfXavxMazECCYilLNNOw%3D%3D"
+			(at 218.44 99.06 0)
+			(hide yes)
+			(show_name no)
+			(do_not_autoplace no)
+			(effects
+				(font
+					(size 1.27 1.27)
+				)
+			)
+		)
+		(property "Mouser Part Number" "https://www.mouser.com/en/ProductDetail/Vishay-Draloric/RCS04021K00FKED?qs=NKmfXavxMazECCYilLNNOw%3D%3D"
+			(at 218.44 99.06 0)
+			(hide yes)
+			(show_name no)
+			(do_not_autoplace no)
+			(effects
+				(font
+					(size 1.27 1.27)
+				)
+			)
+		)
+		(property "Manufacturer_Part_Number" "RCS04021K00FKED"
+			(at 218.44 99.06 0)
+			(hide yes)
+			(show_name no)
+			(do_not_autoplace no)
+			(effects
+				(font
+					(size 1.27 1.27)
+				)
+			)
+		)
+		(property "Manufacturer_Name" "Vishay / Draloric"
 			(at 218.44 99.06 0)
 			(hide yes)
@@
 			)
 		)
-		(property "Datasheet" "https://www.mouser.com/ProductDetail/Vishay-Beyschlag/MCS04020C1001FE000?qs=sGAEpiMZZMtlubZbdhIBIMFZrYW9%252Bak7nVRDfe1Ameo%3D"
+		(property "Datasheet" "https://www.mouser.com/en/ProductDetail/Vishay-Draloric/RCS04021K00FKED?qs=NKmfXavxMazECCYilLNNOw%3D%3D"
+			(at 233.68 33.02 0)
+			(hide yes)
+			(show_name no)
+			(do_not_autoplace no)
+			(effects
+				(font
+					(size 1.27 1.27)
+				)
+			)
+		)
+		(property "Mouser Part Number" "https://www.mouser.com/en/ProductDetail/Vishay-Draloric/RCS04021K00FKED?qs=NKmfXavxMazECCYilLNNOw%3D%3D"
+			(at 233.68 33.02 0)
+			(hide yes)
+			(show_name no)
+			(do_not_autoplace no)
+			(effects
+				(font
+					(size 1.27 1.27)
+				)
+			)
+		)
+		(property "Manufacturer_Part_Number" "RCS04021K00FKED"
+			(at 233.68 33.02 0)
+			(hide yes)
+			(show_name no)
+			(do_not_autoplace no)
+			(effects
+				(font
+					(size 1.27 1.27)
+				)
+			)
+		)
+		(property "Manufacturer_Name" "Vishay / Draloric"
 			(at 233.68 33.02 0)
 			(hide yes)

Commit message: add a unit test fixture, and start changing the current measurement circuit
Connections:
- net fault renamed mainFault
- no-connect marks 0 -> 14
Changed lines of the file:
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@@
 		(color 0 0 0 0)
 	)
+	(no_connect
+		(at 172.72 59.69)
+	)
+	(no_connect
+		(at 127 92.71)
+	)
+	(no_connect
+		(at 127 49.53)
+	)
+	(no_connect
+		(at 149.86 31.75)
+	)
+	(no_connect
+		(at 127 46.99)
+	)
+	(no_connect
+		(at 172.72 64.77)
+	)
+	(no_connect
+		(at 172.72 67.31)
+	)
+	(no_connect
+		(at 172.72 72.39)
+	)
+	(no_connect
+		(at 172.72 57.15)
+	)
+	(no_connect
+		(at 172.72 62.23)
+	)
+	(no_connect
+		(at 127 90.17)
+	)
+	(no_connect
+		(at 144.78 31.75)
+	)
+	(no_connect
+		(at 127 87.63)
+	)
+	(no_connect
+		(at 172.72 69.85)
+	)
 	(wire
 		(pts
@@
 		)
 	)
-	(label "fault"
+	(label "mainFault"
 		(at 114.3 80.01 0)
 		(effects
@@
 		)
 	)
-	(label "fault"
+	(label "mainFault"
 		(at 201.93 77.47 0)
 		(effects
@@
 			)
 		)
-		(property "Mouser Part Number" "https://www.mouser.com/en/ProductDetail/Vishay-Draloric/RCS04021K00FKED?qs=NKmfXavxMazECCYilLNNOw%3D%3D"
+		(property "Description" "Resistor"
 			(at 218.44 72.39 0)
 			(hide yes)
@@
 			)
 		)
-		(property "Manufacturer_Part_Number" "RCS04021K00FKED"
+		(property "Mouser Part Number" "https://www.mouser.com/en/ProductDetail/Vishay-Draloric/RCS04021K00FKED?qs=NKmfXavxMazECCYilLNNOw%3D%3D"
 			(at 218.44 72.39 0)
 			(hide yes)
@@
 			)
 		)
-		(property "Manufacturer_Name" "Vishay / Draloric"
+		(property "Manufacturer_Part_Number" "RCS04021K00FKED"
 			(at 218.44 72.39 0)
 			(hide yes)
@@
 			)
 		)
-		(property "Description" "Resistor"
+		(property "Manufacturer_Name" "Vishay / Draloric"
 			(at 218.44 72.39 0)
 			(hide yes)
@@
 			)
 		)
-		(property "Mouser Part Number" "https://www.mouser.com/en/ProductDetail/Vishay-Draloric/RCS04021K00FKED?qs=NKmfXavxMazECCYilLNNOw%3D%3D"
+		(property "Description" "Resistor"
 			(at 218.44 99.06 0)
 			(hide yes)
@@
 			)
 		)
-		(property "Manufacturer_Part_Number" "RCS04021K00FKED"
+		(property "Mouser Part Number" "https://www.mouser.com/en/ProductDetail/Vishay-Draloric/RCS04021K00FKED?qs=NKmfXavxMazECCYilLNNOw%3D%3D"
 			(at 218.44 99.06 0)
 			(hide yes)
@@
 			)
 		)
-		(property "Manufacturer_Name" "Vishay / Draloric"
+		(property "Manufacturer_Part_Number" "RCS04021K00FKED"
 			(at 218.44 99.06 0)
 			(hide yes)
@@
 			)
 		)
-		(property "Description" "Resistor"
+		(property "Manufacturer_Name" "Vishay / Draloric"
 			(at 218.44 99.06 0)
 			(hide yes)
@@
 			)
 		)
-		(property "Mouser Part Number" "https://www.mouser.com/en/ProductDetail/Vishay-Draloric/RCS04021K00FKED?qs=NKmfXavxMazECCYilLNNOw%3D%3D"
+		(property "Description" "Resistor"
 			(at 233.68 33.02 0)
 			(hide yes)
@@
 			)
 		)
-		(property "Manufacturer_Part_Number" "RCS04021K00FKED"
+		(property "Mouser Part Number" "https://www.mouser.com/en/ProductDetail/Vishay-Draloric/RCS04021K00FKED?qs=NKmfXavxMazECCYilLNNOw%3D%3D"
 			(at 233.68 33.02 0)
 			(hide yes)
@@
 			)
 		)
-		(property "Manufacturer_Name" "Vishay / Draloric"
+		(property "Manufacturer_Part_Number" "RCS04021K00FKED"
 			(at 233.68 33.02 0)
 			(hide yes)
@@
 			)
 		)
-		(property "Description" "Resistor"
+		(property "Manufacturer_Name" "Vishay / Draloric"
 			(at 233.68 33.02 0)
 			(hide yes)
