File: mainBoard/MainControler.kicad_sch (KiCad schematic)
At the start: 37 parts, among them J2 Conn_01x10_Pin, J20 1935161, J21 1935161, J22 Conn_01x16_Socket, J23 1935161, J24 1935161, J25 1935161, U13 TCMT1109, U14 TCMT1109, U4 ESP32-S3-DevKitC, U5 SX1509

Commit message: sch update
Connections:
- net 3.3V_Main: now also J22.15 (Pin_15)
- net 5V_Main: now also J22.16 (Pin_16)
- net CLK: now also J22.5 (Pin_5)
- net CS1: now also J22.4 (Pin_4)
- net GND: now also J22.1 (Pin_1), J22.8 (Pin_8)
- net MISO: now also J22.6 (Pin_6)
- net MOSI: now also J22.7 (Pin_7)
- net SCL: now also J22.2 (Pin_2)
- net SDA: now also J22.3 (Pin_3)
- net thermoDrdy_0: now also J22.13 (Pin_13)
- net thermoDrdy_1: now also J22.11 (Pin_11)
- net thermoDrdy_2: now also J22.9 (Pin_9)
- net thermoFault_0: now also J22.14 (Pin_14)
- net thermoFault_1: now also J22.12 (Pin_12)
- net thermoFault_2: now also J22.10 (Pin_10)
Other:
- removed sheet Thermocouple1
- removed sheet Thermocouple2
- removed sheet Thermocouple3
- note added: "Thermocouple Connection"
- moved on the sheet: J22

Commit message: progress
Parts:
- removed J22: Conn_01x16_Socket, Connector_PinSocket_2.54mm:PinSocket_1x16_P2.54mm_Horizontal, symbol Connector:Conn_01x16_Socket
- added J6: Conn_01x20_Socket, symbol Connector:Conn_01x20_Socket
Connections:
- net 3.3V_Main: now also J6.19 (Pin_19)
- net 5V_Main: now also J6.20 (Pin_20)
- net CLK: now also J6.9 (Pin_9)
- net CS0: now also J6.8 (Pin_8)
- net CS1: now also J6.7 (Pin_7)
- net CS2: now also J6.6 (Pin_6)
- net GND: now also J6.1 (Pin_1), J6.12 (Pin_12), J6.2 (Pin_2), J6.3 (Pin_3)
- net MISO: now also J6.10 (Pin_10)
- net MOSI: now also J6.11 (Pin_11)
- net SCL: now also J6.4 (Pin_4)
- net SDA: now also J6.5 (Pin_5)
- net thermoDrdy_0: now also J6.17 (Pin_17)
- net thermoDrdy_1: now also J6.15 (Pin_15)
- net thermoDrdy_2: now also J6.13 (Pin_13)
- net thermoFault_0: now also J6.18 (Pin_18)
- net thermoFault_1: now also J6.16 (Pin_16)
- net thermoFault_2: now also J6.14 (Pin_14)

Commit message: progress
Parts:
- J6: footprint (none) -> Connector_PinSocket_2.54mm:PinSocket_1x20_P2.54mm_Horizontal
Changed lines of the file:
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@@
 			)
 		)
-		(property "Footprint" ""
+		(property "Footprint" "Connector_PinSocket_2.54mm:PinSocket_1x20_P2.54mm_Horizontal"
 			(at 101.6 163.83 0)
 			(hide yes)

Commit message: i think the pcbs and sch are good
Parts:
- R15: Manufacturer_Name (none) -> Vishay / Draloric; Manufacturer_Part_Number (none) -> RCS04021K00FKED; Mouser Part Number (none) -> https://www.mouser.com/en/ProductDetail/Vishay-Draloric/RCS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
Changed lines of the file:
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@@
 			)
 		)
-		(property "Datasheet" "https://www.mouser.com/ProductDetail/Vishay-Beyschlag/MCS04020C1001FE000?qs=sGAEpiMZZMtlubZbdhIBIMFZrYW9%252Bak7nVRDfe1Ameo%3D"
+		(property "Datasheet" "https://www.mouser.com/en/ProductDetail/Vishay-Draloric/RCS04021K00FKED?qs=NKmfXavxMazECCYilLNNOw%3D%3D"
 			(at 250.19 80.01 0)
 			(hide yes)
+			(show_name no)
+			(do_not_autoplace no)
+			(effects
+				(font
+					(size 1.27 1.27)
+				)
+			)
+		)
+		(property "Mouser Part Number" "https://www.mouser.com/en/ProductDetail/Vishay-Draloric/RCS04021K00FKED?qs=NKmfXavxMazECCYilLNNOw%3D%3D"
+			(at 250.19 80.01 0)
+			(hide yes)
+			(show_name no)
+			(do_not_autoplace no)
+			(effects
+				(font
+					(size 1.27 1.27)
+				)
+			)
+		)
+		(property "Manufacturer_Part_Number" "RCS04021K00FKED"
+			(at 250.19 80.01 0)
+			(hide yes)
+			(show_name no)
+			(do_not_autoplace no)
+			(effects
+				(font
+					(size 1.27 1.27)
+				)
+			)
+		)
+		(property "Manufacturer_Name" "Vishay / Draloric"
+			(at 250.19 80.01 0)
+			(hide yes)

Commit message: add a unit test fixture, and start changing the current measurement circuit
Connections:
- no-connect marks 14 -> 22
Changed lines of the file:
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@@
 	)
 	(no_connect
+		(at 218.44 76.2)
+	)
+	(no_connect
 		(at 218.44 66.04)
 	)
@@
 	)
 	(no_connect
+		(at 218.44 81.28)
+	)
+	(no_connect
+		(at 167.64 58.42)
+	)
+	(no_connect
+		(at 167.64 68.58)
+	)
+	(no_connect
 		(at 218.44 132.08)
 	)
@@
 	)
 	(no_connect
+		(at 167.64 66.04)
+	)
+	(no_connect
+		(at 218.44 78.74)
+	)
+	(no_connect
 		(at 218.44 134.62)
 	)
 	(no_connect
+		(at 237.49 241.3)
+	)
+	(no_connect
+		(at 191.77 53.34)
+	)
+	(no_connect
 		(at 219.71 60.96)
 	)
@@
 	(wire
 		(pts
+			(xy 73.66 251.46) (xy 77.47 251.46)
+		)
+		(stroke
+			(width 0)
+			(type default)
+		)
+	)
+	(wire
+		(pts
 			(xy 218.44 86.36) (xy 255.27 86.36)
 		)
@@
 	(wire
 		(pts
-			(xy 73.66 251.46) (xy 77.47 251.46)
-		)
-		(stroke
-			(width 0)
-			(type default)
-		)
-	)
-	(wire
-		(pts
 			(xy 355.6 177.8) (xy 355.6 179.07)
 		)
@@
 	(wire
 		(pts
+			(xy 73.66 254) (xy 73.66 251.46)
+		)
+		(stroke
+			(width 0)
+			(type default)
+		)
+	)
+	(wire
+		(pts
 			(xy 106.68 179.07) (xy 111.76 179.07)
 		)
@@
 	(wire
 		(pts
-			(xy 73.66 254) (xy 73.66 251.46)
-		)
-		(stroke
-			(width 0)
-			(type default)
-		)
-	)
-	(wire
-		(pts
 			(xy 218.44 91.44) (xy 255.27 91.44)
 		)
@@
 			)
 		)
-		(property "Mouser Part Number" "https://www.mouser.com/en/ProductDetail/Vishay-Draloric/RCS04021K00FKED?qs=NKmfXavxMazECCYilLNNOw%3D%3D"
+		(property "Description" "Resistor"
 			(at 250.19 80.01 0)
 			(hide yes)
@@
 			)
 		)
-		(property "Manufacturer_Part_Number" "RCS04021K00FKED"
+		(property "Mouser Part Number" "https://www.mouser.com/en/ProductDetail/Vishay-Draloric/RCS04021K00FKED?qs=NKmfXavxMazECCYilLNNOw%3D%3D"
 			(at 250.19 80.01 0)
 			(hide yes)
@@
 			)
 		)
-		(property "Manufacturer_Name" "Vishay / Draloric"
+		(property "Manufacturer_Part_Number" "RCS04021K00FKED"
 			(at 250.19 80.01 0)
 			(hide yes)
@@
 			)
 		)
-		(property "Description" "Resistor"
+		(property "Manufacturer_Name" "Vishay / Draloric"
 			(at 250.19 80.01 0)
 			(hide yes)
@@
 		)
 	)
-	(group ""
-		(members "01d73998-251e-46de-a2fb-a5a766ac558a" "0573eaf9-e3df-4530-962c-78bc83545154"
-			"0737ef3c-69a1-468c-8842-02ca677120c3" "117851f6-d39b-4fea-8490-fd64b189ec0f"
-			"11c982a4-99ba-45fc-834c-d547e334d636" "1389095e-d52a-4619-af64-e9910dc7c62e"
-			"1ec62650-1534-4460-b805-bf7b33f4c68d" "244220b5-df49-43ee-a84f-561544e6ed67"
-			"2916a857-e3b9-44ed-bde1-e73f86681a16" "2cce3e1d-ccf5-4310-9af2-4968b5e5e0b5"
-			"303affac-7630-4324-aca9-6191ae359fd5" "33ecd58f-5c1f-4b58-b38a-0af34679d267"
-			"345ba1de-b0bb-4ef3-a095-0c0381bd9f19" "3610133e-be30-44a0-abe6-0374ff26957c"
-			"4de58580-80ba-4376-9790-77f9885ee922" "63fd10b0-d1e2-4439-9774-1a8b257597a7"
-			"6724e6ac-942f-45c6-b0f2-1750c4c1cf61" "6bf8ce12-cc33-4862-905e-dd1731657d5b"
-			"6e13c2b5-94ac-4a6c-8c8e-c6d59b729331" "6f9be0ac-ca73-4f51-b23b-16a67ae84d74"
-			"751c634f-5138-4078-9bd3-a79a12005d8d" "79cb8098-5fc5-49db-9993-ad819d0f9bb4"
-			"848a709c-d019-45d1-8bfa-23270ccef253" "84b57c7d-5f05-4494-8b27-49d0c0f12979"
-			"8fcc2f90-6476-4ce6-9dcc-8fe79655140f" "96dde035-5b41-42e1-bc7b-e5b832ca1820"
-			"98406b61-8a98-4104-84d1-7287adea4546" "a84bf762-754e-45cd-8956-712b8932ab94"
-			"b35f2077-1983-439a-b7c7-ba24ba265ea4" "b545b762-d2df-4408-bdc4-224515640d70"
-			"bf66c716-06dc-4d7d-9e17-9c4a2297bbb9" "c3f3c1c7-367d-41cd-b6cf-4467d28b0b73"
-			"cb40a6e9-53fc-44d5-8f34-a1f8bf702a5c" "dfe1a20b-0dda-4c17-abd3-430b66453aaf"
-			"e5f57a7b-d976-41bf-87c8-a6a07491b757" "f45116ee-173d-4db6-934d-32365a809670"
-			"f88bfe89-8103-4f8f-8378-326cad5fa3a3"
-		)
-	)

Commit message: note that rgb led must be removed from esp32
Other:
- note added: "Must REMOVE RGB LED. FOR THERMOFAULT 0/2 to work"
Changed lines of the file:
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@@
+		)
+	)
+	(text "Must REMOVE RGB LED. FOR THERMOFAULT 0/2 to work"
+		(exclude_from_sim no)
+		(at 263.906 136.906 0)
+		(effects
+			(font
+				(size 1.27 1.27)
+			)
 		)
 	)
