File: SaftyThermocoupleBoard/ThermocoupleBoard.kicad_sch (KiCad schematic)
At the start: 8 parts, among them J5 Conn_01x20_Pin, U1 LT1962-3.3

Commit message: add single thermocouple board
Parts:
- removed J5: Conn_01x20_Pin, Connector_PinHeader_2.54mm:PinHeader_1x20_P2.54mm_Horizontal, symbol Connector:Conn_01x20_Pin
- added J1: Conn_02x06_Odd_Even, Connector_PinHeader_2.54mm:PinHeader_2x06_P2.54mm_Horizontal, symbol Connector_Generic:Conn_02x06_Odd_Even
Connections:
- net 5V: now also J1.2 (Pin_2)
- net CLK: now also J1.9 (Pin_9)
- net CS0: now also J1.11 (Pin_11)
- net GND: now also J1.10 (Pin_10), J1.12 (Pin_12)
- net MISO: now also J1.7 (Pin_7)
- net MOSI: now also J1.5 (Pin_5)
- net SCL: now also J1.8 (Pin_8)
- net SDA: now also J1.6 (Pin_6)
- net thermoDrdy_0: now also J1.4 (Pin_4)
- net thermoFault_0: now also J1.3 (Pin_3)
- net at R2.2: now also J1.1 (Pin_1)
Other:
- removed sheet Thermocouple2
- removed sheet Thermocouple3
- moved on the sheet: C1, C2, C28, C3, R1, R2, U1

Commit message: mainboard pcb changes for jlc pcb dfm
Parts:
- J1: footprint Connector_PinHeader_2.54mm:PinHeader_2x06_P2.54mm_Horizontal -> Connector_PinHeader_1.27mm:PinHeader_2x06_P1.27mm_Horizontal
Changed lines of the file:
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@@
 			)
 		)
-		(property "Footprint" "Connector_PinHeader_2.54mm:PinHeader_2x06_P2.54mm_Horizontal"
+		(property "Footprint" "Connector_PinHeader_1.27mm:PinHeader_2x06_P1.27mm_Horizontal"
 			(at 229.87 120.65 0)
 			(hide yes)
