File: UnitTest/UnitTestFixture.kicad_sch (KiCad schematic)
At the start: 3 parts, among them U1 ESP32-S3-DevKitC, U2 AD9833xRM, U3 MCP4728

Commit message: kiln fw update
Parts:
- added U4, U5: PCF8575DBR, Package_SO:SSOP-24_5.3x8.2mm_P0.65mm, symbol Interface_Expansion:PCF8575DBR
Connections:
- net SCL: now also U4.22 (SCL), U5.22 (SCL)
- net SDA: now also U4.23 (SDA), U5.23 (SDA)
- net Expander_IRQ_1: now reaches U1.10 (GPIO17/ADC2_CH6)
- net Expander_IRQ_1: now also U5.1 (~{INT})
- net Expander_IRQ_0: now reaches U1.11 (GPIO18/ADC2_CH7)
- net Expander_IRQ_0: now also U4.1 (~{INT})
- net GND: now reaches U1.22 (GND), U1.23 (GND), U1.24 (GND), U1.44 (GND)
- net GND: now also U4.12 (GND), U4.2 (A1), U4.21 (A0), U4.3 (A2), U5.12 (GND), U5.2 (A1), U5.3 (A2)
- new net VCC: U4.24 (VCC), U5.21 (A0), U5.24 (VCC)
